File: 1300-watts-RMS-for-4-ohms-class-TD-audio-power-amp-DEV-4/OVERLOAD_PROTECTOR.kicad_sch (KiCad schematic)
At the start: 47 parts, among them Q901 2N5401, Q902 2N5551, Q903 TIP41C, U901 RC4558

Commit message: Update Sun Sep 11 07:00:26 PM WIB 2022
Other:
- company: (none) -> BSD POWER AMP
Changed lines of the file:
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@@
     (title "1300 WATTS RMS CLASS-TD\\nAUDIO POWER AMPLIFIER\\nFOR 4-OHMS LOUDSPEAKER")
     (date "2022-09-11")
+    (company "BSD POWER AMP")
   )
   (junction (at 57.15 31.75) (diameter 0) (color 0 0 0 0)

Commit message: Update Mon Sep 12 10:35:28 AM WIB 2022
Parts:
- C901, C902, C903, C904: footprint MATRIX_1.4:CAPACITOR_AE_D7.62mm -> BSD_POWER_AMP:CAPACITOR_AE_D7.62mm
- CNT406, CNT407: footprint MATRIX_1.4:SOLDER-TAB-6.3-mm -> BSD_POWER_AMP:SOLDER-TAB-6.3-mm
- D901, D903: footprint MATRIX_1.4:DIODE_ZENER_AXIAL_SMALL_SI -> BSD_POWER_AMP:DIODE_ZENER_AXIAL_SMALL_SI; symbol MATRIX_1.4:D_Zener -> BSD_POWER_AMP:D_Zener
- D902, D904, D905, D906, D907, D908, D909, D910, D911, D912, D913: footprint MATRIX_1.4:DIODE_AXIAL_SMALL_GE -> BSD_POWER_AMP:DIODE_AXIAL_SMALL_GE; symbol MATRIX_1.4:D -> BSD_POWER_AMP:D
- D914: footprint MATRIX_1.4:DIODE_AXIAL_SMALL_SI -> BSD_POWER_AMP:DIODE_AXIAL_SMALL_SI; symbol MATRIX_1.4:D -> BSD_POWER_AMP:D
- D915: symbol MATRIX_1.4:LED -> BSD_POWER_AMP:LED
- Q901: footprint MATRIX_1.4:TO-92-EBC -> BSD_POWER_AMP:TO-92-EBC; symbol MATRIX_1.4:Q_PNP_CBE -> BSD_POWER_AMP:Q_PNP_CBE
- Q902: footprint MATRIX_1.4:TO-92-EBC -> BSD_POWER_AMP:TO-92-EBC; symbol MATRIX_1.4:Q_NPN_CBE -> BSD_POWER_AMP:Q_NPN_CBE
- Q903: footprint MATRIX_1.4:TO-220 -> BSD_POWER_AMP:TO-220; symbol MATRIX_1.4:Q_NPN_CBE -> BSD_POWER_AMP:Q_NPN_CBE
- R901, R902, R903, R904, R905, R906, R908, R909, R910, R911, R912, R913, R914, R915, R917: footprint MATRIX_1.4:RESISTOR_AXIAL_0.25W -> BSD_POWER_AMP:RESISTOR_AXIAL_0.25W
- R907, R916: footprint MATRIX_1.4:RESISTOR_AXIAL_0.5W -> BSD_POWER_AMP:RESISTOR_AXIAL_0.5W
- S901: footprint MATRIX_1.4:Relay_SPDT_RAYEX-L90 -> BSD_POWER_AMP:Relay_SPDT_RAYEX-L90; symbol MATRIX_1.4:RAYEX-L90A -> BSD_POWER_AMP:RAYEX-L90A
- U901: footprint MATRIX_1.4:DIP8 -> BSD_POWER_AMP:DIP8
