File: 1300-watts-RMS-for-4-ohms-class-TD-audio-power-amp-DEV-4/OVERLOAD_PROTECTOR.kicad_sch (KiCad schematic)
At the start: 47 parts, among them Q901 2N5401, Q902 2N5551, Q903 TIP41C, U901 RC4558

Commit message: Update Wed Sep 14 11:14:32 AM WIB 2022
Other:
- moved on the sheet: C901, C902, C903, C904, CNT406, CNT407, CNT901, CNT902, CNT903, CNT904, D901, D902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

Commit message: Update Sat Sep 17 07:48:27 PM WIB 2022
Parts:
- D901, D903: footprint BSD_POWER_AMP:DIODE_ZENER_AXIAL_SMALL_SI -> BSD_POWER_AMP:D_DO-41_SOD81_P10.16mm_Zener_Horizontal
- D902, D904, D905, D906, D907, D908, D909, D910, D911, D912, D913: footprint BSD_POWER_AMP:DIODE_AXIAL_SMALL_GE -> BSD_POWER_AMP:D_DO-35_SOD27_P10.16mm_Horizontal
- D914: footprint BSD_POWER_AMP:DIODE_AXIAL_SMALL_SI -> BSD_POWER_AMP:D_DO-41_SOD81_P10.16mm_Horizontal
- Q901, Q902: footprint BSD_POWER_AMP:TO-92-EBC -> BSD_POWER_AMP:TO-92_Inline_Wide_EBC
- R901, R902, R903, R904, R905, R906, R908, R909, R910, R911, R912, R913, R914, R915, R917: footprint BSD_POWER_AMP:RESISTOR_AXIAL_0.25W -> BSD_POWER_AMP:R_Axial_DIN0207_L6.3mm_D2.5mm_P10.16mm_Horizontal
- R907, R916: footprint BSD_POWER_AMP:RESISTOR_AXIAL_0.5W -> BSD_POWER_AMP:R_Axial_DIN0309_L9.0mm_D3.2mm_P12.70mm_Horizontal

Commit message: Update Sat Sep 17 09:34:05 PM WIB 2022
Parts:
- U901: footprint BSD_POWER_AMP:DIP8 -> BSD_POWER_AMP:DIP-8_W7.62mm
Connections:
- net -15V: now also R914.2; no longer R914.1
- net 0: now also R908.2, R909.2, R911.2; no longer R908.1, R909.1, R911.1
- net PTC_OP: now also R916.1; no longer R916.2
- net PTC_REF: now also R914.1, R915.2; no longer R914.2, R915.1
- net at D908.1 (A), D909.2 (K), R906.2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: now also R911.1; no longer R911.2
- net at D907.1 (A), D908.2 (K), U901.1: now also R910.1; no longer R910.2
- net at C903.1, D905.1 (A), D906.2 (K)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: now also R908.1; no longer R908.2
- net at D911.2 (K): now also R915.1; no longer R915.2
- net at D913.2 (K), Q903.2 (B): now also R916.2; no longer R916.1
- new net: R909.1, R910.2, U901.2 (-)
Changed lines of the file:
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@@
     (pin "1")
   )
-  (symbol (lib_id "Device:R") (at 114.3 68.58 180) (unit 1)
+  (symbol (lib_name "R_9") (lib_id "Device:R") (at 114.3 68.58 0) (mirror y) (unit 1)
     (in_bom yes) (on_board yes)
     (property "Reference" "R909" (id 0) (at 120.65 66.04 0))
@@
     (pin "2")
   )
-  (symbol (lib_id "Device:R") (at 133.35 43.18 180) (unit 1)
+  (symbol (lib_id "Device:R") (at 133.35 43.18 0) (mirror y) (unit 1)
     (in_bom yes) (on_board yes)
     (property "Reference" "R911" (id 0) (at 139.7 40.64 0))
@@
     (pin "2")
   )
-  (symbol (lib_id "Device:R") (at 69.85 43.18 180) (unit 1)
+  (symbol (lib_name "R_1") (lib_id "Device:R") (at 69.85 43.18 180) (unit 1)
     (in_bom yes) (on_board yes)
     (property "Reference" "R905" (id 0) (at 76.2 40.64 0))
@@
     (pin "2")
   )
-  (symbol (lib_id "Device:R") (at 158.75 113.03 90) (unit 1)
+  (symbol (lib_name "R_12") (lib_id "Device:R") (at 158.75 113.03 90) (unit 1)
     (in_bom yes) (on_board yes)
     (property "Reference" "R913" (id 0) (at 158.75 116.84 90))
@@
     (pin "2")
   )
-  (symbol (lib_id "Device:R") (at 88.9 74.93 90) (unit 1)
+  (symbol (lib_name "R_5") (lib_id "Device:R") (at 88.9 74.93 90) (unit 1)
     (in_bom yes) (on_board yes)
     (property "Reference" "R907" (id 0) (at 88.9 78.74 90))
@@
     (pin "2")
   )
-  (symbol (lib_id "Device:R") (at 107.95 81.28 180) (unit 1)
+  (symbol (lib_name "R_8") (lib_id "Device:R") (at 107.95 81.28 0) (mirror y) (unit 1)
     (in_bom yes) (on_board yes)
     (property "Reference" "R908" (id 0) (at 114.3 78.74 0))
@@
     (pin "2")
   )
-  (symbol (lib_id "Device:R") (at 114.3 36.83 90) (unit 1)
+  (symbol (lib_name "R_6") (lib_id "Device:R") (at 114.3 36.83 90) (unit 1)
     (in_bom yes) (on_board yes)
     (property "Reference" "R906" (id 0) (at 114.3 40.64 90))
@@
     (property "Reference" "U901" (id 0) (at 124.46 44.45 0))
     (property "Value" "RC4558" (id 1) (at 124.46 46.99 0))
-    (property "Footprint" "BSD_POWER_AMP:DIP8" (id 2) (at 127 54.61 0)
+    (property "Footprint" "BSD_POWER_AMP:DIP-8_W7.62mm" (id 2) (at 127 54.61 0)
       (effects (font (size 1.27 1.27)) hide)
     )
@@
     (pin "1")
   )
-  (symbol (lib_id "Device:R") (at 133.35 62.23 90) (unit 1)
+  (symbol (lib_name "R_10") (lib_id "Device:R") (at 133.35 62.23 270) (mirror x) (unit 1)
     (in_bom yes) (on_board yes)
     (property "Reference" "R910" (id 0) (at 133.35 66.04 90))
@@
     (pin "2")
   )
-  (symbol (lib_id "Device:R") (at 222.25 81.28 90) (unit 1)
+  (symbol (lib_name "R_15") (lib_id "Device:R") (at 222.25 81.28 90) (unit 1)
     (in_bom yes) (on_board yes)
     (property "Reference" "R917" (id 0) (at 222.25 85.09 90))
@@
     (pin "2")
   )
-  (symbol (lib_id "Device:R") (at 146.05 113.03 90) (unit 1)
+  (symbol (lib_name "R_11") (lib_id "Device:R") (at 146.05 113.03 90) (unit 1)
     (in_bom yes) (on_board yes)
     (property "Reference" "R912" (id 0) (at 146.05 116.84 90))
@@
     (pin "2")
   )
-  (symbol (lib_id "Device:R") (at 190.5 55.88 180) (unit 1)
+  (symbol (lib_name "R_16") (lib_id "Device:R") (at 190.5 55.88 0) (mirror y) (unit 1)
     (in_bom yes) (on_board yes)
     (property "Reference" "R916" (id 0) (at 196.85 53.34 0))
@@
     (pin "3")
   )
-  (symbol (lib_id "Device:R") (at 158.75 100.33 90) (unit 1)
+  (symbol (lib_name "R_13") (lib_id "Device:R") (at 158.75 100.33 270) (mirror x) (unit 1)
     (in_bom yes) (on_board yes)
     (property "Reference" "R914" (id 0) (at 158.75 104.14 90))
@@
     (property "Reference" "U901" (id 0) (at 114.3 156.21 0))
     (property "Value" "RC4558" (id 1) (at 114.3 158.75 0))
-    (property "Footprint" "BSD_POWER_AMP:DIP8" (id 2) (at 110.49 157.48 0)
+    (property "Footprint" "BSD_POWER_AMP:DIP-8_W7.62mm" (id 2) (at 110.49 157.48 0)
       (effects (font (size 1.27 1.27)) hide)
     )
@@
     (property "Reference" "U901" (id 0) (at 179.07 53.34 0))
     (property "Value" "RC4558" (id 1) (at 179.07 55.88 0))
-    (property "Footprint" "BSD_POWER_AMP:DIP8" (id 2) (at 179.07 45.72 0)
+    (property "Footprint" "BSD_POWER_AMP:DIP-8_W7.62mm" (id 2) (at 179.07 45.72 0)
       (effects (font (size 1.27 1.27)) hide)
     )
@@
     (pin "1")
   )
-  (symbol (lib_id "Device:R") (at 69.85 93.98 180) (unit 1)
+  (symbol (lib_name "R_3") (lib_id "Device:R") (at 69.85 93.98 180) (unit 1)
     (in_bom yes) (on_board yes)
     (property "Reference" "R901" (id 0) (at 76.2 91.44 0))
@@
     (pin "2")
   )
-  (symbol (lib_id "Device:R") (at 114.3 93.98 90) (unit 1)
+  (symbol (lib_name "R_7") (lib_id "Device:R") (at 114.3 93.98 90) (unit 1)
     (in_bom yes) (on_board yes)
     (property "Reference" "R903" (id 0) (at 114.3 97.79 90))
@@
     (pin "1")
   )
-  (symbol (lib_id "Device:R") (at 171.45 81.28 90) (unit 1)
+  (symbol (lib_name "R_14") (lib_id "Device:R") (at 171.45 81.28 270) (mirror x) (unit 1)
     (in_bom yes) (on_board yes)
     (property "Reference" "R915" (id 0) (at 171.45 85.09 90))
@@
     (pin "2")
   )
-  (symbol (lib_id "Device:R") (at 69.85 106.68 180) (unit 1)
+  (symbol (lib_name "R_4") (lib_id "Device:R") (at 69.85 106.68 180) (unit 1)
     (in_bom yes) (on_board yes)
     (property "Reference" "R902" (id 0) (at 76.2 104.14 0))
@@
     (pin "2")
   )
-  (symbol (lib_id "Device:R") (at 69.85 55.88 180) (unit 1)
+  (symbol (lib_name "R_2") (lib_id "Device:R") (at 69.85 55.88 180) (unit 1)
     (in_bom yes) (on_board yes)
     (property "Reference" "R904" (id 0) (at 76.2 53.34 0))

Commit message: Update Mon Sep 19 08:13:41 AM WIB 2022
Parts:
- C901, C902, C904: footprint BSD_POWER_AMP:CAPACITOR_AE_D7.62mm -> BSD_POWER_AMP:CP_Radial_D5.0mm_P2.00mm
- C903: footprint BSD_POWER_AMP:CAPACITOR_AE_D7.62mm -> BSD_POWER_AMP:CP_Radial_D8.0mm_P3.50mm
- Q903: footprint BSD_POWER_AMP:TO-220 -> BSD_POWER_AMP:TO-220-3_Vertical
Changed lines of the file:
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@@
     (property "Reference" "C902" (id 0) (at 127 161.29 0))
     (property "Value" "47uF" (id 1) (at 127 163.83 0))
-    (property "Footprint" "BSD_POWER_AMP:CAPACITOR_AE_D7.62mm" (id 2) (at 121.6152 167.64 0)
+    (property "Footprint" "BSD_POWER_AMP:CP_Radial_D5.0mm_P2.00mm" (id 2) (at 121.6152 167.64 0)
       (effects (font (size 1.27 1.27)) hide)
     )
@@
     (property "Reference" "Q903" (id 0) (at 209.55 60.96 0))
     (property "Value" "TIP41C" (id 1) (at 209.55 63.5 0))
-    (property "Footprint" "BSD_POWER_AMP:TO-220" (id 2) (at 205.74 59.69 0)
+    (property "Footprint" "BSD_POWER_AMP:TO-220-3_Vertical" (id 2) (at 205.74 59.69 0)
       (effects (font (size 1.27 1.27)) hide)
     )
@@
     (property "Reference" "C904" (id 0) (at 209.55 85.09 90))
     (property "Value" "10uF" (id 1) (at 209.55 87.63 90))
-    (property "Footprint" "BSD_POWER_AMP:CAPACITOR_AE_D7.62mm" (id 2) (at 205.74 82.2452 0)
+    (property "Footprint" "BSD_POWER_AMP:CP_Radial_D5.0mm_P2.00mm" (id 2) (at 205.74 82.2452 0)
       (effects (font (size 1.27 1.27)) hide)
     )
@@
     (property "Reference" "C901" (id 0) (at 127 148.59 0))
     (property "Value" "47uF" (id 1) (at 127 151.13 0))
-    (property "Footprint" "BSD_POWER_AMP:CAPACITOR_AE_D7.62mm" (id 2) (at 121.6152 154.94 0)
+    (property "Footprint" "BSD_POWER_AMP:CP_Radial_D5.0mm_P2.00mm" (id 2) (at 121.6152 154.94 0)
       (effects (font (size 1.27 1.27)) hide)
     )
@@
     (property "Reference" "C903" (id 0) (at 101.6 78.74 0))
     (property "Value" "220uF" (id 1) (at 101.6 81.28 0))
-    (property "Footprint" "BSD_POWER_AMP:CAPACITOR_AE_D7.62mm" (id 2) (at 96.2152 85.09 0)
-      (effects (font (size 1.27 1.27)) hide)
-    )
+    (property "Footprint" "BSD_POWER_AMP:CP_Radial_D8.0mm_P3.50mm" (id 2) (at 96.2152 85.09 0)
+      (effects (font (size 1.27 1.27)) hide)
+    )

Commit message: Update Mon Sep 19 09:56:34 AM WIB 2022
Parts:
- D901, D903: footprint BSD_POWER_AMP:D_DO-41_SOD81_P10.16mm_Zener_Horizontal -> BSD_POWER_AMP:D_T-1_P10.16mm_Zener_Horizontal
Changed lines of the file:
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@@
     (property "Reference" "D901" (id 0) (at 76.2 80.01 90))
     (property "Value" "1N4734" (id 1) (at 76.2 82.55 90))
-    (property "Footprint" "BSD_POWER_AMP:D_DO-41_SOD81_P10.16mm_Zener_Horizontal" (id 2) (at 69.85 81.28 0)
+    (property "Footprint" "BSD_POWER_AMP:D_T-1_P10.16mm_Zener_Horizontal" (id 2) (at 69.85 81.28 0)
       (effects (font (size 1.27 1.27)) hide)
     )
@@
     (property "Reference" "D903" (id 0) (at 76.2 67.31 90))
     (property "Value" "1N4734" (id 1) (at 76.2 69.85 90))
-    (property "Footprint" "BSD_POWER_AMP:D_DO-41_SOD81_P10.16mm_Zener_Horizontal" (id 2) (at 69.85 68.58 0)
-      (effects (font (size 1.27 1.27)) hide)
-    )
+    (property "Footprint" "BSD_POWER_AMP:D_T-1_P10.16mm_Zener_Horizontal" (id 2) (at 69.85 68.58 0)
+      (effects (font (size 1.27 1.27)) hide)
+    )

Commit message: Update Sat Sep 24 09:59:01 AM WIB 2022
Changed lines of the file:
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@@
   (title_block
     (title "1300 WATTS RMS CLASS-TD\\nAUDIO POWER AMPLIFIER\\nFOR 4-OHMS LOUDSPEAKER")
-    (date "2022-09-14")
+    (date "2022-09-24")
     (company "BSD POWER AMP")
   )

Commit message: Update Sun Sep 25 11:43:47 AM WIB 2022
Parts:
- CNT406, CNT407: value Solder Tab 6.3 mm -> Solder_Tab_W6.35mm_P5.08mm; footprint BSD_POWER_AMP:SOLDER-TAB-6.3-mm -> BSD_POWER_AMP:Solder_Tab_W6.35mm_P5.08mm
Changed lines of the file:
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@@
     (in_bom yes) (on_board yes)
     (property "Reference" "CNT407" (id 0) (at 279.4 66.04 0))
-    (property "Value" "Solder Tab 6.3 mm" (id 1) (at 279.4 58.42 0)
+    (property "Value" "Solder_Tab_W6.35mm_P5.08mm" (id 1) (at 279.4 58.42 0)
       (effects (font (size 1.27 1.27)) hide)
     )
-    (property "Footprint" "BSD_POWER_AMP:SOLDER-TAB-6.3-mm" (id 2) (at 279.4 62.23 0)
+    (property "Footprint" "BSD_POWER_AMP:Solder_Tab_W6.35mm_P5.08mm" (id 2) (at 279.4 62.23 0)
       (effects (font (size 1.27 1.27)) hide)
     )
@@
     (in_bom yes) (on_board yes)
     (property "Reference" "CNT406" (id 0) (at 279.4 40.64 0))
-    (property "Value" "Solder Tab 6.3 mm" (id 1) (at 279.4 33.02 0)
+    (property "Value" "Solder_Tab_W6.35mm_P5.08mm" (id 1) (at 279.4 33.02 0)
       (effects (font (size 1.27 1.27)) hide)
     )
-    (property "Footprint" "BSD_POWER_AMP:SOLDER-TAB-6.3-mm" (id 2) (at 279.4 36.83 0)
+    (property "Footprint" "BSD_POWER_AMP:Solder_Tab_W6.35mm_P5.08mm" (id 2) (at 279.4 36.83 0)
       (effects (font (size 1.27 1.27)) hide)
     )
