File: 1300-watts-RMS-for-4-ohms-class-TD-audio-power-amp-DEV-4/POWER-AMP-BLOCK.kicad_sch (KiCad schematic)
At the start: 169 parts, among them Q401 MPSA42, Q402 MPSA42, Q403 MPSA92, Q404 MPSA92, Q405 MJE340, Q406 MJE350, Q407 MJE350, Q408 MJE340, Q409 MJE15032, Q410 MJE15033, Q411 2SC5200, Q412 2SA1943, Q4131 2SC5200, Q4132 2SC5200, Q4133 2SC5200, Q4134 2SC5200, Q4135 2SC5200, Q4136 2SC5200, Q4141 2SA1943, Q4142 2SA1943, Q4143 2SA1943, Q4144 2SA1943, Q4145 2SA1943, Q4146 2SA1943, Q601 2N5401, Q602 MJE340, Q603 MJE340, Q604 MJE15032, Q605 2SC5200, Q606 2N5401, Q607 2N5401, Q608 2N5401, Q609 MJE350, Q610 2N5551, Q611 MJE340, Q701 2N5551, Q702 MJE350, Q703 MJE350, Q704 MJE15033, Q705 2SA1943, Q706 2N5551, Q707 2N5551, Q708 2N5401, Q709 MJE350, Q710 2N5551, Q711 MJE340

Commit message: Update Sun Sep 11 07:00:26 PM WIB 2022
Other:
- company: (none) -> BSD POWER AMP
Changed lines of the file:
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@@
     (title "1300 WATTS RMS CLASS-TD\\nAUDIO POWER AMPLIFIER\\nFOR 4-OHMS LOUDSPEAKER")
     (date "2022-09-11")
+    (company "BSD POWER AMP")
   )
   (junction (at 234.95 107.95) (diameter 0) (color 0 0 0 0)

Commit message: Update Mon Sep 12 10:35:28 AM WIB 2022
Parts:
- C401: footprint MATRIX_1.4:CAPACITOR_AE_D7.62mm -> BSD_POWER_AMP:CAPACITOR_AE_D7.62mm
- C402, C404: footprint MATRIX_1.4:CAPACITOR_CERAMIC_STD -> BSD_POWER_AMP:CAPACITOR_CERAMIC_STD
- C403, C408, C410, C601, C701: footprint MATRIX_1.4:CAPACITOR_AE_D10mm -> BSD_POWER_AMP:CAPACITOR_AE_D10mm
- C405, C406, C407, C409: footprint MATRIX_1.4:0.1uF_250V_Vishay_Roederstein_MKT_1822 -> BSD_POWER_AMP:0.1uF_250V_Vishay_Roederstein_MKT_1822
- C602, C702: footprint MATRIX_1.4:CAPACITOR_CERAMIC_LEAD_PITCH_7.62mm -> BSD_POWER_AMP:CAPACITOR_CERAMIC_LEAD_PITCH_7.62mm
- C603, C703: footprint MATRIX_1.4:0.0022uF_400V_Vishay_Roederstein_MKT_1822 -> BSD_POWER_AMP:0.0022uF_400V_Vishay_Roederstein_MKT_1822
- C604, C704: footprint MATRIX_1.4:1uF_250V_Vishay_Roederstein_MKT_1822 -> BSD_POWER_AMP:1uF_250V_Vishay_Roederstein_MKT_1822
- CNT403, CNT404, CNT405: footprint MATRIX_1.4:SOLDER-TAB-6.3-mm -> BSD_POWER_AMP:SOLDER-TAB-6.3-mm
- D401: footprint MATRIX_1.4:DIODE_AXIAL_SMALL_SI -> BSD_POWER_AMP:DIODE_AXIAL_SMALL_SI; symbol MATRIX_1.4:D_Zener -> BSD_POWER_AMP:D_Zener
- D601, D602, D604, D606, D610, D701, D702, D704, D706, D709: footprint MATRIX_1.4:DIODE_AXIAL_SMALL_SI -> BSD_POWER_AMP:DIODE_AXIAL_SMALL_SI; symbol MATRIX_1.4:D -> BSD_POWER_AMP:D
- D603, D605, D609, D611, D703, D705, D710: footprint MATRIX_1.4:DIODE_ZENER_AXIAL_SMALL_SI -> BSD_POWER_AMP:DIODE_ZENER_AXIAL_SMALL_SI; symbol MATRIX_1.4:D_Zener -> BSD_POWER_AMP:D_Zener
- D607, D608, D614, D707, D708: footprint MATRIX_1.4:DIODE_POWER_TO-220AC -> BSD_POWER_AMP:DIODE_POWER_TO-220AC; symbol MATRIX_1.4:D -> BSD_POWER_AMP:D
- D612, D613, D615, D711, D712, D713, D714: footprint MATRIX_1.4:DIODE_POWER_TO-220AC-MIRRORED -> BSD_POWER_AMP:DIODE_POWER_TO-220AC-MIRRORED; symbol MATRIX_1.4:D -> BSD_POWER_AMP:D
- L401: footprint MATRIX_1.4:INDUCTOR_AIR_CORE_3uH_D600mils_L750mils -> BSD_POWER_AMP:INDUCTOR_AIR_CORE_3uH_D600mils_L750mils
- L601, L701: footprint MATRIX_1.4:TOROIDAL_INDUCTOR_0077083A7 -> BSD_POWER_AMP:TOROIDAL_INDUCTOR_0077083A7
- Q401, Q402, Q610, Q701, Q706, Q707, Q710: footprint MATRIX_1.4:TO-92-EBC -> BSD_POWER_AMP:TO-92-EBC; symbol MATRIX_1.4:Q_NPN_CBE -> BSD_POWER_AMP:Q_NPN_CBE
- Q403, Q404, Q601, Q606, Q607, Q608, Q708: footprint MATRIX_1.4:TO-92-EBC -> BSD_POWER_AMP:TO-92-EBC; symbol MATRIX_1.4:Q_PNP_CBE -> BSD_POWER_AMP:Q_PNP_CBE
- Q405, Q408, Q602, Q603, Q611, Q711: footprint MATRIX_1.4:TO-225 -> BSD_POWER_AMP:TO-225; symbol MATRIX_1.4:Q_NPN_CBE -> BSD_POWER_AMP:Q_NPN_CBE
- Q406, Q407, Q609, Q702, Q703, Q709: footprint MATRIX_1.4:TO-225 -> BSD_POWER_AMP:TO-225; symbol MATRIX_1.4:Q_PNP_CBE -> BSD_POWER_AMP:Q_PNP_CBE
- Q409, Q604: footprint MATRIX_1.4:TO-220-MIRRORED -> BSD_POWER_AMP:TO-220-MIRRORED; symbol MATRIX_1.4:Q_NPN_CBE -> BSD_POWER_AMP:Q_NPN_CBE
- Q410, Q704: footprint MATRIX_1.4:TO-220-MIRRORED -> BSD_POWER_AMP:TO-220-MIRRORED; symbol MATRIX_1.4:Q_PNP_CBE -> BSD_POWER_AMP:Q_PNP_CBE
- Q411, Q4131, Q4132, Q4133, Q4134, Q4135, Q4136, Q605: footprint MATRIX_1.4:TO-264-MIRRORED -> BSD_POWER_AMP:TO-264-MIRRORED; symbol MATRIX_1.4:Q_NPN_CBE -> BSD_POWER_AMP:Q_NPN_CBE
- Q412, Q4141, Q4142, Q4143, Q4144, Q4145, Q4146, Q705: footprint MATRIX_1.4:TO-264-MIRRORED -> BSD_POWER_AMP:TO-264-MIRRORED; symbol MATRIX_1.4:Q_PNP_CBE -> BSD_POWER_AMP:Q_PNP_CBE
- R401, R4041, R4051, R4052, R4061, R4062, R4071, R4072, R4073, R4074, R4081, R4082, R4091, R4092, R410, R411, R412, R413, R4141, R4142, R608, R708, RG401: footprint MATRIX_1.4:RESISTOR_AXIAL_0.25W -> BSD_POWER_AMP:RESISTOR_AXIAL_0.25W
- R4021, R4031, R4151, R601, R602, R603, R604, R605, R606, R611, R612, R701, R702, R703, R704, R705, R706, R711: footprint MATRIX_1.4:RESISTOR_AXIAL_0.5W -> BSD_POWER_AMP:RESISTOR_AXIAL_0.5W
- R4161, R4171, R4181, R4182, R4183, R4184, R4185, R4186, R4191, R4192, R4193, R4194, R4195, R4196, R420, R607, R707: footprint MATRIX_1.4:RESISTOR_BLOCK_5W -> BSD_POWER_AMP:RESISTOR_BLOCK_5W
- R609, R610, R709, R710: footprint MATRIX_1.4:RESISTOR_AXIAL_2W -> BSD_POWER_AMP:RESISTOR_AXIAL_2W
- RT401: footprint MATRIX_1.4:RESISTOR_ROUND_TRIMPOT_STD -> BSD_POWER_AMP:RESISTOR_ROUND_TRIMPOT_STD
- XQ6011, XQ6012, XQ7011, XQ7012: footprint MATRIX_1.4:TO-264-MIRRORED -> BSD_POWER_AMP:TO-264-MIRRORED; symbol MATRIX_1.4:Q_NMOS_DGS -> BSD_POWER_AMP:Q_NMOS_DGS

Commit message: Update Mon Sep 12 03:35:30 PM WIB 2022
Connections:
- net VSLDRVP: now also D610.2 (K), Q608.2 (B), R611.2
Changed lines of the file:
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@@
   (junction (at 368.3 57.15) (diameter 0) (color 0 0 0 0)
+  )
+  (junction (at 266.7 57.15) (diameter 0) (color 0 0 0 0)
   )
   (junction (at 146.05 19.05) (diameter 0) (color 0 0 0 0)
@@
     (stroke (width 0) (type default) (color 0 0 0 0))
   )
+  (wire (pts (xy 266.7 57.15) (xy 266.7 78.74))
+    (stroke (width 0) (type default) (color 0 0 0 0))
+  )
   (wire (pts (xy 228.6 101.6) (xy 228.6 109.22))
     (stroke (width 0) (type default) (color 0 0 0 0))
@@
     (stroke (width 0) (type default) (color 0 0 0 0))
   )
-  (wire (pts (xy 266.7 55.88) (xy 266.7 78.74))
+  (wire (pts (xy 266.7 55.88) (xy 266.7 57.15))
     (stroke (width 0) (type default) (color 0 0 0 0))
   )
@@
     (stroke (width 0) (type default) (color 0 0 0 0))
   )
+  (wire (pts (xy 266.7 57.15) (xy 279.4 57.15))
+    (stroke (width 0) (type default) (color 0 0 0 0))
+  )
