File: 1300-watts-RMS-for-4-ohms-class-TD-audio-power-amp-DEV-4/POWER-AMP-BLOCK.kicad_sch (KiCad schematic)
At the start: 169 parts, among them Q401 MPSA42, Q402 MPSA42, Q403 MPSA92, Q404 MPSA92, Q405 MJE340, Q406 MJE350, Q407 MJE350, Q408 MJE340, Q409 MJE15032, Q410 MJE15033, Q411 2SC5200, Q412 2SA1943, Q4131 2SC5200, Q4132 2SC5200, Q4133 2SC5200, Q4134 2SC5200, Q4135 2SC5200, Q4136 2SC5200, Q4141 2SA1943, Q4142 2SA1943, Q4143 2SA1943, Q4144 2SA1943, Q4145 2SA1943, Q4146 2SA1943, Q601 2N5401, Q602 MJE340, Q603 MJE340, Q604 MJE15032, Q605 2SC5200, Q606 2N5401, Q607 2N5401, Q608 2N5401, Q609 MJE350, Q610 2N5551, Q611 MJE340, Q701 2N5551, Q702 MJE350, Q703 MJE350, Q704 MJE15033, Q705 2SA1943, Q706 2N5551, Q707 2N5551, Q708 2N5401, Q709 MJE350, Q710 2N5551, Q711 MJE340

Commit message: Update Wed Sep 14 11:14:32 AM WIB 2022
Parts:
- added D711: BAV21, BSD_POWER_AMP:DIODE_AXIAL_SMALL_SI, symbol BSD_POWER_AMP:D
- C404: footprint BSD_POWER_AMP:CAPACITOR_CERAMIC_STD -> BSD_POWER_AMP:CAPACITOR_CERAMIC_LEAD_PITCH_7.62mm
- R4021: footprint BSD_POWER_AMP:RESISTOR_AXIAL_0.5W -> BSD_POWER_AMP:RESISTOR_AXIAL_0.25W; Wattage 0.5W -> 0.25W
- R4071, R4072, R4073, R4074: footprint BSD_POWER_AMP:RESISTOR_AXIAL_0.25W -> BSD_POWER_AMP:RESISTOR_AXIAL_0.5W
- renumbered D711 to D712, D712 to D713, D713 to D714, D714 to D715
Connections:
- net VSFN: now also D711.2 (K)
- net VSGZN: now also D711.1 (A)
Changed lines of the file:
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@@
   (title_block
     (title "1300 WATTS RMS CLASS-TD\\nAUDIO POWER AMPLIFIER\\nFOR 4-OHMS LOUDSPEAKER")
-    (date "2022-09-13")
+    (date "2022-09-14")
     (company "BSD POWER AMP")
   )
@@
   (junction (at 254 101.6) (diameter 0) (color 0 0 0 0)
   )
+  (junction (at 304.8 190.5) (diameter 0) (color 0 0 0 0)
+  )
   (junction (at 120.65 57.15) (diameter 0) (color 0 0 0 0)
   )
@@
     (stroke (width 0) (type default) (color 0 0 0 0))
   )
+  (wire (pts (xy 302.26 190.5) (xy 304.8 190.5))
+    (stroke (width 0) (type default) (color 0 0 0 0))
+  )
   (polyline (pts (xy 45.72 251.46) (xy 45.72 15.24))
     (stroke (width 0) (type default) (color 0 0 0 0))
@@
     (stroke (width 0) (type default) (color 0 0 0 0))
   )
+  (wire (pts (xy 292.1 190.5) (xy 292.1 196.85))
+    (stroke (width 0) (type default) (color 0 0 0 0))
+  )
   (wire (pts (xy 304.8 120.65) (xy 323.85 120.65))
     (stroke (width 0) (type default) (color 0 0 0 0))
@@
     (stroke (width 0) (type default) (color 0 0 0 0))
   )
+  (wire (pts (xy 294.64 190.5) (xy 292.1 190.5))
+    (stroke (width 0) (type default) (color 0 0 0 0))
+  )
   (polyline (pts (xy 336.55 165.1) (xy 336.55 101.6))
     (stroke (width 0) (type dash) (color 0 0 0 0))
@@
     (pin "2")
   )
+  (symbol (lib_id "BSD_POWER_AMP:D") (at 298.45 190.5 0) (mirror y) (unit 1)
+    (in_bom yes) (on_board yes)
+    (property "Reference" "D711" (id 0) (at 298.45 182.88 0))
+    (property "Value" "BAV21" (id 1) (at 298.45 185.42 0))
+    (property "Footprint" "BSD_POWER_AMP:DIODE_AXIAL_SMALL_SI" (id 2) (at 298.45 190.5 0)
+      (effects (font (size 1.27 1.27)) hide)
+    )
+    (property "Datasheet" "~" (id 3) (at 298.45 190.5 0)
+      (effects (font (size 1.27 1.27)) hide)
+    )
+    (property "Spice_Primitive" "D" (id 4) (at 299.72 214.63 0)
+      (effects (font (size 1.27 1.27)) hide)
+    )
+    (property "Spice_Model" "1N4007" (id 5) (at 297.18 214.63 0)
+      (effects (font (size 1.27 1.27)) hide)
+    )
+    (property "Spice_Netlist_Enabled" "Y" (id 6) (at 302.26 214.63 0)
+      (effects (font (size 1.27 1.27)) hide)
+    )
+    (property "Spice_Lib_File" "spice_models/model.lib" (id 7) (at 294.64 214.63 0)
+      (effects (font (size 1.27 1.27)) hide)
+    )
+    (pin "1")
+    (pin "2")
+  )
   (symbol (lib_id "pspice:0") (at 50.8 177.8 0) (unit 1)
     (in_bom yes) (on_board yes)
@@
     (property "Reference" "R4021" (id 0) (at 57.15 67.31 90))
     (property "Value" "22k" (id 1) (at 57.15 69.85 90))
-    (property "Footprint" "BSD_POWER_AMP:RESISTOR_AXIAL_0.5W" (id 2) (at 57.15 74.422 90)
+    (property "Footprint" "BSD_POWER_AMP:RESISTOR_AXIAL_0.25W" (id 2) (at 57.15 74.422 90)
       (effects (font (size 1.27 1.27)) hide)
     )
@@
       (effects (font (size 1.27 1.27)) hide)
     )
-    (property "Wattage" "0.5W" (id 4) (at 57.15 72.39 90))
+    (property "Wattage" "0.25W" (id 4) (at 57.15 72.39 90))
     (pin "1")
     (pin "2")
@@
   (symbol (lib_id "BSD_POWER_AMP:D") (at 393.7 222.25 90) (mirror x) (unit 1)
     (in_bom yes) (on_board yes)
-    (property "Reference" "D714" (id 0) (at 398.78 222.25 0))
+    (property "Reference" "D715" (id 0) (at 398.78 222.25 0))
     (property "Value" "MURF1560" (id 1) (at 401.32 222.25 0))
     (property "Footprint" "BSD_POWER_AMP:DIODE_POWER_TO-220AC-MIRRORED" (id 2) (at 393.7 222.25 0)
@@
     (property "Reference" "R4074" (id 0) (at 101.6 194.31 90))
     (property "Value" "82k" (id 1) (at 101.6 196.85 90))
-    (property "Footprint" "BSD_POWER_AMP:RESISTOR_AXIAL_0.25W" (id 2) (at 101.6 204.978 90)
+    (property "Footprint" "BSD_POWER_AMP:RESISTOR_AXIAL_0.5W" (id 2) (at 101.6 204.978 90)
       (effects (font (size 1.27 1.27)) hide)
     )
@@
     (property "Reference" "R4073" (id 0) (at 101.6 181.61 90))
     (property "Value" "82k" (id 1) (at 101.6 184.15 90))
-    (property "Footprint" "BSD_POWER_AMP:RESISTOR_AXIAL_0.25W" (id 2) (at 101.6 192.278 90)
+    (property "Footprint" "BSD_POWER_AMP:RESISTOR_AXIAL_0.5W" (id 2) (at 101.6 192.278 90)
       (effects (font (size 1.27 1.27)) hide)
     )
@@
     (property "Reference" "R4072" (id 0) (at 101.6 168.91 90))
     (property "Value" "82k" (id 1) (at 101.6 171.45 90))
-    (property "Footprint" "BSD_POWER_AMP:RESISTOR_AXIAL_0.25W" (id 2) (at 101.6 179.578 90)
+    (property "Footprint" "BSD_POWER_AMP:RESISTOR_AXIAL_0.5W" (id 2) (at 101.6 179.578 90)
       (effects (font (size 1.27 1.27)) hide)
     )
@@
   (symbol (lib_id "BSD_POWER_AMP:D") (at 368.3 184.15 90) (mirror x) (unit 1)
     (in_bom yes) (on_board yes)
-    (property "Reference" "D711" (id 0) (at 360.68 184.15 0))
+    (property "Reference" "D712" (id 0) (at 360.68 184.15 0))
     (property "Value" "MURF1560" (id 1) (at 363.22 184.15 0))
     (property "Footprint" "BSD_POWER_AMP:DIODE_POWER_TO-220AC-MIRRORED" (id 2) (at 368.3 184.15 0)
@@
   (symbol (lib_id "BSD_POWER_AMP:D") (at 368.3 222.25 90) (mirror x) (unit 1)
     (in_bom yes) (on_board yes)
-    (property "Reference" "D712" (id 0) (at 373.38 222.25 0))
+    (property "Reference" "D713" (id 0) (at 373.38 222.25 0))
     (property "Value" "MURF1560" (id 1) (at 375.92 222.25 0))
     (property "Footprint" "BSD_POWER_AMP:DIODE_POWER_TO-220AC-MIRRORED" (id 2) (at 368.3 222.25 0)
@@
     (property "Reference" "R4071" (id 0) (at 101.6 156.21 90))
     (property "Value" "82k" (id 1) (at 101.6 158.75 90))
-    (property "Footprint" "BSD_POWER_AMP:RESISTOR_AXIAL_0.25W" (id 2) (at 101.6 166.878 90)
+    (property "Footprint" "BSD_POWER_AMP:RESISTOR_AXIAL_0.5W" (id 2) (at 101.6 166.878 90)
       (effects (font (size 1.27 1.27)) hide)
     )
@@
     (property "Reference" "C404" (id 0) (at 127 48.26 90))
     (property "Value" "220pF" (id 1) (at 127 50.8 90))
-    (property "Footprint" "BSD_POWER_AMP:CAPACITOR_CERAMIC_STD" (id 2) (at 130.81 56.1848 0)
+    (property "Footprint" "BSD_POWER_AMP:CAPACITOR_CERAMIC_LEAD_PITCH_7.62mm" (id 2) (at 130.81 56.1848 0)
       (effects (font (size 1.27 1.27)) hide)
     )
@@
   (symbol (lib_id "BSD_POWER_AMP:D") (at 381 165.1 90) (mirror x) (unit 1)
     (in_bom yes) (on_board yes)
-    (property "Reference" "D713" (id 0) (at 386.08 165.1 0))
+    (property "Reference" "D714" (id 0) (at 386.08 165.1 0))
     (property "Value" "MURF1560" (id 1) (at 388.62 165.1 0))
     (property "Footprint" "BSD_POWER_AMP:DIODE_POWER_TO-220AC-MIRRORED" (id 2) (at 381 165.1 0)

Commit message: Update Wed Sep 14 04:55:10 PM WIB 2022
Parts:
- D401: footprint BSD_POWER_AMP:DIODE_AXIAL_SMALL_SI -> BSD_POWER_AMP:DIODE_ZENER_AXIAL_SMALL_SI
Changed lines of the file:
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@@
     (property "Reference" "D401" (id 0) (at 114.3 240.03 90))
     (property "Value" "1N4730" (id 1) (at 114.3 242.57 90))
-    (property "Footprint" "BSD_POWER_AMP:DIODE_AXIAL_SMALL_SI" (id 2) (at 107.95 241.3 0)
+    (property "Footprint" "BSD_POWER_AMP:DIODE_ZENER_AXIAL_SMALL_SI" (id 2) (at 107.95 241.3 0)
       (effects (font (size 1.27 1.27)) hide)
     )

Commit message: Update Sat Sep 17 07:48:27 PM WIB 2022
Parts:
- C402: footprint BSD_POWER_AMP:CAPACITOR_CERAMIC_STD -> BSD_POWER_AMP:C_Disc_D8.0mm_W5.0mm_P10.00mm
- C404, C602, C702: footprint BSD_POWER_AMP:CAPACITOR_CERAMIC_LEAD_PITCH_7.62mm -> BSD_POWER_AMP:C_Disc_D8.0mm_W5.0mm_P10.00mm
- C405, C406, C407, C409: footprint BSD_POWER_AMP:0.1uF_250V_Vishay_Roederstein_MKT_1822 -> BSD_POWER_AMP:C_Rect_L18.0mm_W6.0mm_P15.00mm_FKS3_FKP3
- C604, C704: footprint BSD_POWER_AMP:1uF_250V_Vishay_Roederstein_MKT_1822 -> BSD_POWER_AMP:C_Rect_L26.5mm_W8.5mm_P22.50mm_MKS4
- D401, D603, D605, D609, D611, D703, D705, D710: footprint BSD_POWER_AMP:DIODE_ZENER_AXIAL_SMALL_SI -> BSD_POWER_AMP:D_DO-41_SOD81_P10.16mm_Zener_Horizontal
- D601, D604, D606, D701, D704, D706: footprint BSD_POWER_AMP:DIODE_AXIAL_SMALL_SI -> BSD_POWER_AMP:D_DO-41_SOD81_P10.16mm_Horizontal
- D602, D610, D702, D709, D711: footprint BSD_POWER_AMP:DIODE_AXIAL_SMALL_SI -> BSD_POWER_AMP:D_DO-35_SOD27_P10.16mm_Horizontal
- Q401, Q402, Q403, Q404, Q601, Q606, Q607, Q608, Q610, Q701, Q706, Q707, Q708, Q710: footprint BSD_POWER_AMP:TO-92-EBC -> BSD_POWER_AMP:TO-92_Inline_Wide_EBC
- R401, R4021, R4041, R4051, R4052, R4061, R4062, R4081, R4082, R4091, R4092, R410, R411, R412, R413, R4141, R4142, R608, R708, RG401: footprint BSD_POWER_AMP:RESISTOR_AXIAL_0.25W -> BSD_POWER_AMP:R_Axial_DIN0207_L6.3mm_D2.5mm_P10.16mm_Horizontal
- R4031, R4071, R4072, R4073, R4074, R4151, R601, R602, R603, R604, R605, R606, R611, R612, R701, R702, R703, R704, R705, R706, R711: footprint BSD_POWER_AMP:RESISTOR_AXIAL_0.5W -> BSD_POWER_AMP:R_Axial_DIN0309_L9.0mm_D3.2mm_P12.70mm_Horizontal
- R4161, R4171, R4181, R4182, R4183, R4184, R4185, R4186, R4191, R4192, R4193, R4194, R4195, R4196, R420, R607, R707: footprint BSD_POWER_AMP:RESISTOR_BLOCK_5W -> BSD_POWER_AMP:R_Axial_Shunt_L22.2mm_W9.5mm_PS14.30mm_P25.40mm
- R609, R610, R709, R710: footprint BSD_POWER_AMP:RESISTOR_AXIAL_2W -> BSD_POWER_AMP:R_Axial_DIN0516_L15.5mm_D5.0mm_P20.32mm_Horizontal
Connections:
- net +120V: now also C407.1, C602.1; no longer C407.2, C602.2
- net -120V: now also C409.2, C702.2; no longer C409.1, C702.1
- net 0: now also C406.2, C407.2, C409.1, C604.2, C704.1, R703.1, R709.1, R710.1; no longer C406.1, C407.1, C409.2, C604.1, C704.2, R703.2, R709.2, R710.2
- net DIFF_P: now also C404.2; no longer C404.1
- net DRVN1: now also R4151.2; no longer R4151.1
- net DRVN2: now also R4171.2; no longer R4171.1
- net DRVP1: now also R4151.1; no longer R4151.2
- net DRVP2: now also R4161.1; no longer R4161.2
- net INPUT_GND: now also R4021.1; no longer R4021.2
- net REF: now also R4021.2; no longer R4021.1
- net VASN: now also C405.2; no longer C405.1
- net VASP: now also C404.1, C405.1, R411.1; no longer C404.2, C405.2, R411.2
- net VMOUT: now also R4161.2, R4171.1; no longer R4161.1, R4171.2
- net VSAVN: now also C704.2; no longer C704.1
- net VSAVP: now also C603.2, C604.1; no longer C603.1, C604.2
- net VSFN: now also R711.2; no longer R711.1
- net VSGZN: now also R710.2; no longer R710.1
- net VSGZP: now also R611.2; no longer R611.1
- net VSLDRVP: now also R611.1; no longer R611.2
- net VSTAN: now also R709.2; no longer R709.1
- net VSTCP: now also R608.2; no longer R608.1
- net VSZPN: now also R711.1; no longer R711.2
- net VSZPP: now also C603.1; no longer C603.2
- net at D603.2 (K), Q602.2 (B), R602.2: now also C602.2; no longer C602.1
- net at C701.1, D702.1 (A), Q701.2 (B): now also R703.2; no longer R703.1
- net at Q606.2 (B): now also R608.1; no longer R608.2
- net at R420.2: now also C406.1; no longer C406.2
- net at D703.1 (A), Q702.2 (B): now also C702.1, R702.1; no longer C702.2, R702.2
- net at Q407.2 (B), R410.1, R412.2: now also R411.2; no longer R411.1
- net at C701.2, D701.1 (A): now also R702.2; no longer R702.1

Commit message: Update Sat Sep 17 10:08:16 PM WIB 2022
Parts:
- Q405, Q406, Q408, Q602, Q603, Q609, Q611, Q702, Q703, Q709, Q711: footprint BSD_POWER_AMP:TO-225 -> BSD_POWER_AMP:TO-126-3_Vertical
- Q407: footprint BSD_POWER_AMP:TO-225 -> BSD_POWER_AMP:TO-126-3_Vertical_For_Bottom_Layer
Changed lines of the file:
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@@
     (property "Reference" "Q408" (id 0) (at 139.7 214.63 0))
     (property "Value" "MJE340" (id 1) (at 139.7 217.17 0))
-    (property "Footprint" "BSD_POWER_AMP:TO-225" (id 2) (at 135.89 213.36 0)
+    (property "Footprint" "BSD_POWER_AMP:TO-126-3_Vertical" (id 2) (at 135.89 213.36 0)
       (effects (font (size 1.27 1.27)) hide)
     )
@@
     (property "Reference" "Q405" (id 0) (at 76.2 214.63 0))
     (property "Value" "MJE340" (id 1) (at 76.2 217.17 0))
-    (property "Footprint" "BSD_POWER_AMP:TO-225" (id 2) (at 80.01 213.36 0)
+    (property "Footprint" "BSD_POWER_AMP:TO-126-3_Vertical" (id 2) (at 80.01 213.36 0)
       (effects (font (size 1.27 1.27)) hide)
     )
@@
     (property "Reference" "Q406" (id 0) (at 139.7 43.18 0))
     (property "Value" "MJE350" (id 1) (at 139.7 45.72 0))
-    (property "Footprint" "BSD_POWER_AMP:TO-225" (id 2) (at 135.89 46.99 0)
+    (property "Footprint" "BSD_POWER_AMP:TO-126-3_Vertical" (id 2) (at 135.89 46.99 0)
       (effects (font (size 1.27 1.27)) hide)
     )
@@
     (property "Reference" "Q709" (id 0) (at 323.85 214.63 0))
     (property "Value" "MJE350" (id 1) (at 323.85 217.17 0))
-    (property "Footprint" "BSD_POWER_AMP:TO-225" (id 2) (at 320.04 218.44 0)
+    (property "Footprint" "BSD_POWER_AMP:TO-126-3_Vertical" (id 2) (at 320.04 218.44 0)
       (effects (font (size 1.27 1.27)) hide)
     )
@@
     (property "Reference" "Q407" (id 0) (at 127 144.78 0))
     (property "Value" "MJE350" (id 1) (at 127 147.32 0))
-    (property "Footprint" "BSD_POWER_AMP:TO-225" (id 2) (at 123.19 148.59 0)
+    (property "Footprint" "BSD_POWER_AMP:TO-126-3_Vertical_For_Bottom_Layer" (id 2) (at 123.19 148.59 0)
       (effects (font (size 1.27 1.27)) hide)
     )
@@
     (property "Reference" "Q703" (id 0) (at 215.9 220.98 0))
     (property "Value" "MJE350" (id 1) (at 215.9 223.52 0))
-    (property "Footprint" "BSD_POWER_AMP:TO-225" (id 2) (at 212.09 224.79 0)
+    (property "Footprint" "BSD_POWER_AMP:TO-126-3_Vertical" (id 2) (at 212.09 224.79 0)
       (effects (font (size 1.27 1.27)) hide)
     )
@@
     (property "Reference" "Q611" (id 0) (at 323.85 36.83 0))
     (property "Value" "MJE340" (id 1) (at 323.85 39.37 0))
-    (property "Footprint" "BSD_POWER_AMP:TO-225" (id 2) (at 320.04 35.56 0)
+    (property "Footprint" "BSD_POWER_AMP:TO-126-3_Vertical" (id 2) (at 320.04 35.56 0)
       (effects (font (size 1.27 1.27)) hide)
     )
@@
     (property "Reference" "Q603" (id 0) (at 215.9 43.18 0))
     (property "Value" "MJE340" (id 1) (at 215.9 45.72 0))
-    (property "Footprint" "BSD_POWER_AMP:TO-225" (id 2) (at 212.09 41.91 0)
+    (property "Footprint" "BSD_POWER_AMP:TO-126-3_Vertical" (id 2) (at 212.09 41.91 0)
       (effects (font (size 1.27 1.27)) hide)
     )
@@
     (property "Reference" "Q702" (id 0) (at 190.5 220.98 0))
     (property "Value" "MJE350" (id 1) (at 190.5 223.52 0))
-    (property "Footprint" "BSD_POWER_AMP:TO-225" (id 2) (at 186.69 224.79 0)
+    (property "Footprint" "BSD_POWER_AMP:TO-126-3_Vertical" (id 2) (at 186.69 224.79 0)
       (effects (font (size 1.27 1.27)) hide)
     )
@@
     (property "Reference" "Q609" (id 0) (at 323.85 49.53 0))
     (property "Value" "MJE350" (id 1) (at 323.85 52.07 0))
-    (property "Footprint" "BSD_POWER_AMP:TO-225" (id 2) (at 320.04 53.34 0)
+    (property "Footprint" "BSD_POWER_AMP:TO-126-3_Vertical" (id 2) (at 320.04 53.34 0)
       (effects (font (size 1.27 1.27)) hide)
     )
@@
     (property "Reference" "Q602" (id 0) (at 190.5 43.18 0))
     (property "Value" "MJE340" (id 1) (at 190.5 45.72 0))
-    (property "Footprint" "BSD_POWER_AMP:TO-225" (id 2) (at 186.69 41.91 0)
+    (property "Footprint" "BSD_POWER_AMP:TO-126-3_Vertical" (id 2) (at 186.69 41.91 0)
       (effects (font (size 1.27 1.27)) hide)
     )
@@
     (property "Reference" "Q711" (id 0) (at 323.85 201.93 0))
     (property "Value" "MJE340" (id 1) (at 323.85 204.47 0))
-    (property "Footprint" "BSD_POWER_AMP:TO-225" (id 2) (at 320.04 200.66 0)
+    (property "Footprint" "BSD_POWER_AMP:TO-126-3_Vertical" (id 2) (at 320.04 200.66 0)
       (effects (font (size 1.27 1.27)) hide)
     )
