File: 1300-watts-RMS-for-4-ohms-class-TD-audio-power-amp-DEV-4/POWER-AMP-BLOCK.kicad_sch (KiCad schematic)
At the start: 170 parts, among them Q401 MPSA42, Q402 MPSA42, Q403 MPSA92, Q404 MPSA92, Q405 MJE340, Q406 MJE350, Q407 MJE350, Q408 MJE340, Q409 MJE15032, Q410 MJE15033, Q411 2SC5200, Q412 2SA1943, Q4131 2SC5200, Q4132 2SC5200, Q4133 2SC5200, Q4134 2SC5200, Q4135 2SC5200, Q4136 2SC5200, Q4141 2SA1943, Q4142 2SA1943, Q4143 2SA1943, Q4144 2SA1943, Q4145 2SA1943, Q4146 2SA1943, Q601 2N5401, Q602 MJE340, Q603 MJE340, Q604 MJE15032, Q605 2SC5200, Q606 2N5401, Q607 2N5401, Q608 2N5401, Q609 MJE350, Q610 2N5551, Q611 MJE340, Q701 2N5551, Q702 MJE350, Q703 MJE350, Q704 MJE15033, Q705 2SA1943, Q706 2N5551, Q707 2N5551, Q708 2N5401, Q709 MJE350, Q710 2N5551, Q711 MJE340

Commit message: Update Mon Sep 19 08:13:41 AM WIB 2022
Parts:
- C401: footprint BSD_POWER_AMP:CAPACITOR_AE_D7.62mm -> BSD_POWER_AMP:CP_Radial_D5.0mm_P2.00mm
- C403, C408, C410, C601, C701: footprint BSD_POWER_AMP:CAPACITOR_AE_D10mm -> BSD_POWER_AMP:CP_Radial_D10.0mm_P5.00mm
- D607, D608, D614, D707, D708: footprint BSD_POWER_AMP:DIODE_POWER_TO-220AC -> BSD_POWER_AMP:TO-220-2_Vertical
- D612, D613, D615, D712, D713, D715: footprint BSD_POWER_AMP:DIODE_POWER_TO-220AC-MIRRORED -> BSD_POWER_AMP:TO-220-2_Vertical_For_Bottom_Layer
- D714: footprint BSD_POWER_AMP:DIODE_POWER_TO-220AC-MIRRORED -> BSD_POWER_AMP:TO-220-2_Vertical
- Q409, Q410, Q604, Q704: footprint BSD_POWER_AMP:TO-220-MIRRORED -> BSD_POWER_AMP:TO-220-3_Vertical_For_Bottom_Layer
Changed lines of the file:
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@@
     (property "Reference" "Q410" (id 0) (at 139.7 189.23 0))
     (property "Value" "MJE15033" (id 1) (at 139.7 191.77 0))
-    (property "Footprint" "BSD_POWER_AMP:TO-220-MIRRORED" (id 2) (at 148.59 199.39 0)
+    (property "Footprint" "BSD_POWER_AMP:TO-220-3_Vertical_For_Bottom_Layer" (id 2) (at 148.59 199.39 0)
       (effects (font (size 1.27 1.27)) hide)
     )
@@
     (property "Reference" "D715" (id 0) (at 398.78 222.25 0))
     (property "Value" "MURF1560" (id 1) (at 401.32 222.25 0))
-    (property "Footprint" "BSD_POWER_AMP:DIODE_POWER_TO-220AC-MIRRORED" (id 2) (at 393.7 222.25 0)
+    (property "Footprint" "BSD_POWER_AMP:TO-220-2_Vertical_For_Bottom_Layer" (id 2) (at 393.7 222.25 0)
       (effects (font (size 1.27 1.27)) hide)
     )
@@
     (property "Reference" "D612" (id 0) (at 360.68 76.2 0))
     (property "Value" "MURF1560" (id 1) (at 363.22 76.2 0))
-    (property "Footprint" "BSD_POWER_AMP:DIODE_POWER_TO-220AC-MIRRORED" (id 2) (at 368.3 76.2 0)
+    (property "Footprint" "BSD_POWER_AMP:TO-220-2_Vertical_For_Bottom_Layer" (id 2) (at 368.3 76.2 0)
       (effects (font (size 1.27 1.27)) hide)
     )
@@
     (property "Reference" "C601" (id 0) (at 165.1 60.96 0))
     (property "Value" "10uF" (id 1) (at 165.1 63.5 0))
-    (property "Footprint" "BSD_POWER_AMP:CAPACITOR_AE_D10mm" (id 2) (at 159.7152 67.31 0)
+    (property "Footprint" "BSD_POWER_AMP:CP_Radial_D10.0mm_P5.00mm" (id 2) (at 159.7152 67.31 0)
       (effects (font (size 1.27 1.27)) hide)
     )
@@
     (property "Reference" "D708" (id 0) (at 234.95 227.33 0))
     (property "Value" "MURF1560" (id 1) (at 234.95 229.87 0))
-    (property "Footprint" "BSD_POWER_AMP:DIODE_POWER_TO-220AC" (id 2) (at 234.95 234.95 0)
+    (property "Footprint" "BSD_POWER_AMP:TO-220-2_Vertical" (id 2) (at 234.95 234.95 0)
       (effects (font (size 1.27 1.27)) hide)
     )
@@
     (property "Reference" "Q704" (id 0) (at 215.9 195.58 0))
     (property "Value" "MJE15033" (id 1) (at 215.9 198.12 0))
-    (property "Footprint" "BSD_POWER_AMP:TO-220-MIRRORED" (id 2) (at 224.79 205.74 0)
+    (property "Footprint" "BSD_POWER_AMP:TO-220-3_Vertical_For_Bottom_Layer" (id 2) (at 224.79 205.74 0)
       (effects (font (size 1.27 1.27)) hide)
     )
@@
     (property "Reference" "D608" (id 0) (at 234.95 36.83 0))
     (property "Value" "MURF1560" (id 1) (at 234.95 39.37 0))
-    (property "Footprint" "BSD_POWER_AMP:DIODE_POWER_TO-220AC" (id 2) (at 234.95 31.75 0)
+    (property "Footprint" "BSD_POWER_AMP:TO-220-2_Vertical" (id 2) (at 234.95 31.75 0)
       (effects (font (size 1.27 1.27)) hide)
     )
@@
     (property "Reference" "C408" (id 0) (at 69.85 54.61 0))
     (property "Value" "10uF" (id 1) (at 69.85 57.15 0))
-    (property "Footprint" "BSD_POWER_AMP:CAPACITOR_AE_D10mm" (id 2) (at 64.4652 60.96 0)
+    (property "Footprint" "BSD_POWER_AMP:CP_Radial_D10.0mm_P5.00mm" (id 2) (at 64.4652 60.96 0)
       (effects (font (size 1.27 1.27)) hide)
     )
@@
     (property "Reference" "C401" (id 0) (at 69.85 105.41 0))
     (property "Value" "10uF" (id 1) (at 69.85 107.95 0))
-    (property "Footprint" "BSD_POWER_AMP:CAPACITOR_AE_D7.62mm" (id 2) (at 64.4652 104.14 0)
+    (property "Footprint" "BSD_POWER_AMP:CP_Radial_D5.0mm_P2.00mm" (id 2) (at 64.4652 104.14 0)
       (effects (font (size 1.27 1.27)) hide)
     )
@@
     (property "Reference" "D613" (id 0) (at 373.38 38.1 0))
     (property "Value" "MURF1560" (id 1) (at 375.92 38.1 0))
-    (property "Footprint" "BSD_POWER_AMP:DIODE_POWER_TO-220AC-MIRRORED" (id 2) (at 368.3 38.1 0)
+    (property "Footprint" "BSD_POWER_AMP:TO-220-2_Vertical_For_Bottom_Layer" (id 2) (at 368.3 38.1 0)
       (effects (font (size 1.27 1.27)) hide)
     )
@@
     (property "Reference" "Q409" (id 0) (at 139.7 74.93 0))
     (property "Value" "MJE15032" (id 1) (at 139.7 77.47 0))
-    (property "Footprint" "BSD_POWER_AMP:TO-220-MIRRORED" (id 2) (at 148.59 67.31 0)
+    (property "Footprint" "BSD_POWER_AMP:TO-220-3_Vertical_For_Bottom_Layer" (id 2) (at 148.59 67.31 0)
       (effects (font (size 1.27 1.27)) hide)
     )
@@
     (property "Reference" "D615" (id 0) (at 398.78 38.1 0))
     (property "Value" "MURF1560" (id 1) (at 401.32 38.1 0))
-    (property "Footprint" "BSD_POWER_AMP:DIODE_POWER_TO-220AC-MIRRORED" (id 2) (at 393.7 38.1 0)
+    (property "Footprint" "BSD_POWER_AMP:TO-220-2_Vertical_For_Bottom_Layer" (id 2) (at 393.7 38.1 0)
       (effects (font (size 1.27 1.27)) hide)
     )
@@
     (property "Reference" "D614" (id 0) (at 386.08 101.6 0))
     (property "Value" "MURF1560" (id 1) (at 388.62 101.6 0))
-    (property "Footprint" "BSD_POWER_AMP:DIODE_POWER_TO-220AC" (id 2) (at 381 101.6 0)
+    (property "Footprint" "BSD_POWER_AMP:TO-220-2_Vertical" (id 2) (at 381 101.6 0)
       (effects (font (size 1.27 1.27)) hide)
     )
@@
     (property "Reference" "C701" (id 0) (at 165.1 200.66 0))
     (property "Value" "10uF" (id 1) (at 165.1 203.2 0))
-    (property "Footprint" "BSD_POWER_AMP:CAPACITOR_AE_D10mm" (id 2) (at 159.7152 207.01 0)
+    (property "Footprint" "BSD_POWER_AMP:CP_Radial_D10.0mm_P5.00mm" (id 2) (at 159.7152 207.01 0)
       (effects (font (size 1.27 1.27)) hide)
     )
@@
     (property "Reference" "D712" (id 0) (at 360.68 184.15 0))
     (property "Value" "MURF1560" (id 1) (at 363.22 184.15 0))
-    (property "Footprint" "BSD_POWER_AMP:DIODE_POWER_TO-220AC-MIRRORED" (id 2) (at 368.3 184.15 0)
+    (property "Footprint" "BSD_POWER_AMP:TO-220-2_Vertical_For_Bottom_Layer" (id 2) (at 368.3 184.15 0)
       (effects (font (size 1.27 1.27)) hide)
     )
@@
     (property "Reference" "Q604" (id 0) (at 215.9 68.58 0))
     (property "Value" "MJE15032" (id 1) (at 215.9 71.12 0))
-    (property "Footprint" "BSD_POWER_AMP:TO-220-MIRRORED" (id 2) (at 224.79 60.96 0)
+    (property "Footprint" "BSD_POWER_AMP:TO-220-3_Vertical_For_Bottom_Layer" (id 2) (at 224.79 60.96 0)
       (effects (font (size 1.27 1.27)) hide)
     )
@@
     (property "Reference" "C403" (id 0) (at 107.95 92.71 0))
     (property "Value" "220uF" (id 1) (at 107.95 95.25 0))
-    (property "Footprint" "BSD_POWER_AMP:CAPACITOR_AE_D10mm" (id 2) (at 102.5652 99.06 0)
+    (property "Footprint" "BSD_POWER_AMP:CP_Radial_D10.0mm_P5.00mm" (id 2) (at 102.5652 99.06 0)
       (effects (font (size 1.27 1.27)) hide)
     )
@@
     (property "Reference" "D607" (id 0) (at 233.68 25.4 0))
     (property "Value" "MURF1560" (id 1) (at 236.22 25.4 0))
-    (property "Footprint" "BSD_POWER_AMP:DIODE_POWER_TO-220AC" (id 2) (at 228.6 25.4 0)
+    (property "Footprint" "BSD_POWER_AMP:TO-220-2_Vertical" (id 2) (at 228.6 25.4 0)
       (effects (font (size 1.27 1.27)) hide)
     )
@@
     (property "Reference" "C410" (id 0) (at 69.85 226.06 0))
     (property "Value" "10uF" (id 1) (at 69.85 228.6 0))
-    (property "Footprint" "BSD_POWER_AMP:CAPACITOR_AE_D10mm" (id 2) (at 64.4652 232.41 0)
+    (property "Footprint" "BSD_POWER_AMP:CP_Radial_D10.0mm_P5.00mm" (id 2) (at 64.4652 232.41 0)
       (effects (font (size 1.27 1.27)) hide)
     )
@@
     (property "Reference" "D713" (id 0) (at 373.38 222.25 0))
     (property "Value" "MURF1560" (id 1) (at 375.92 222.25 0))
-    (property "Footprint" "BSD_POWER_AMP:DIODE_POWER_TO-220AC-MIRRORED" (id 2) (at 368.3 222.25 0)
+    (property "Footprint" "BSD_POWER_AMP:TO-220-2_Vertical_For_Bottom_Layer" (id 2) (at 368.3 222.25 0)
       (effects (font (size 1.27 1.27)) hide)
     )
@@
     (property "Reference" "D714" (id 0) (at 386.08 165.1 0))
     (property "Value" "MURF1560" (id 1) (at 388.62 165.1 0))
-    (property "Footprint" "BSD_POWER_AMP:DIODE_POWER_TO-220AC-MIRRORED" (id 2) (at 381 165.1 0)
+    (property "Footprint" "BSD_POWER_AMP:TO-220-2_Vertical" (id 2) (at 381 165.1 0)
       (effects (font (size 1.27 1.27)) hide)
     )
@@
     (property "Reference" "D707" (id 0) (at 233.68 241.3 0))
     (property "Value" "MURF1560" (id 1) (at 236.22 241.3 0))
-    (property "Footprint" "BSD_POWER_AMP:DIODE_POWER_TO-220AC" (id 2) (at 228.6 241.3 0)
+    (property "Footprint" "BSD_POWER_AMP:TO-220-2_Vertical" (id 2) (at 228.6 241.3 0)
       (effects (font (size 1.27 1.27)) hide)
     )

Commit message: Update Mon Sep 19 09:56:34 AM WIB 2022
Parts:
- D401, D603, D605, D609, D611, D703, D705, D710: footprint BSD_POWER_AMP:D_DO-41_SOD81_P10.16mm_Zener_Horizontal -> BSD_POWER_AMP:D_T-1_P10.16mm_Zener_Horizontal
Changed lines of the file:
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@@
     (property "Reference" "D603" (id 0) (at 177.8 55.88 90))
     (property "Value" "1N4734" (id 1) (at 177.8 58.42 90))
-    (property "Footprint" "BSD_POWER_AMP:D_DO-41_SOD81_P10.16mm_Zener_Horizontal" (id 2) (at 171.45 57.15 0)
+    (property "Footprint" "BSD_POWER_AMP:D_T-1_P10.16mm_Zener_Horizontal" (id 2) (at 171.45 57.15 0)
       (effects (font (size 1.27 1.27)) hide)
     )
@@
     (property "Reference" "D605" (id 0) (at 203.2 55.88 90))
     (property "Value" "1N4744" (id 1) (at 203.2 58.42 90))
-    (property "Footprint" "BSD_POWER_AMP:D_DO-41_SOD81_P10.16mm_Zener_Horizontal" (id 2) (at 196.85 57.15 0)
+    (property "Footprint" "BSD_POWER_AMP:D_T-1_P10.16mm_Zener_Horizontal" (id 2) (at 196.85 57.15 0)
       (effects (font (size 1.27 1.27)) hide)
     )
@@
     (property "Reference" "D611" (id 0) (at 298.45 43.18 90))
     (property "Value" "1N4742" (id 1) (at 298.45 45.72 90))
-    (property "Footprint" "BSD_POWER_AMP:D_DO-41_SOD81_P10.16mm_Zener_Horizontal" (id 2) (at 292.1 44.45 0)
+    (property "Footprint" "BSD_POWER_AMP:D_T-1_P10.16mm_Zener_Horizontal" (id 2) (at 292.1 44.45 0)
       (effects (font (size 1.27 1.27)) hide)
     )
@@
     (property "Reference" "D401" (id 0) (at 114.3 240.03 90))
     (property "Value" "1N4730" (id 1) (at 114.3 242.57 90))
-    (property "Footprint" "BSD_POWER_AMP:D_DO-41_SOD81_P10.16mm_Zener_Horizontal" (id 2) (at 107.95 241.3 0)
+    (property "Footprint" "BSD_POWER_AMP:D_T-1_P10.16mm_Zener_Horizontal" (id 2) (at 107.95 241.3 0)
       (effects (font (size 1.27 1.27)) hide)
     )
@@
     (property "Reference" "D703" (id 0) (at 177.8 208.28 90))
     (property "Value" "1N4734" (id 1) (at 177.8 210.82 90))
-    (property "Footprint" "BSD_POWER_AMP:D_DO-41_SOD81_P10.16mm_Zener_Horizontal" (id 2) (at 171.45 209.55 0)
+    (property "Footprint" "BSD_POWER_AMP:D_T-1_P10.16mm_Zener_Horizontal" (id 2) (at 171.45 209.55 0)
       (effects (font (size 1.27 1.27)) hide)
     )
@@
     (property "Reference" "D705" (id 0) (at 203.2 208.28 90))
     (property "Value" "1N4744" (id 1) (at 203.2 210.82 90))
-    (property "Footprint" "BSD_POWER_AMP:D_DO-41_SOD81_P10.16mm_Zener_Horizontal" (id 2) (at 196.85 209.55 0)
+    (property "Footprint" "BSD_POWER_AMP:D_T-1_P10.16mm_Zener_Horizontal" (id 2) (at 196.85 209.55 0)
       (effects (font (size 1.27 1.27)) hide)
     )
@@
     (property "Reference" "D609" (id 0) (at 260.35 24.13 90))
     (property "Value" "1N4734" (id 1) (at 260.35 26.67 90))
-    (property "Footprint" "BSD_POWER_AMP:D_DO-41_SOD81_P10.16mm_Zener_Horizontal" (id 2) (at 254 25.4 0)
+    (property "Footprint" "BSD_POWER_AMP:D_T-1_P10.16mm_Zener_Horizontal" (id 2) (at 254 25.4 0)
       (effects (font (size 1.27 1.27)) hide)
     )
@@
     (property "Reference" "D710" (id 0) (at 298.45 208.28 90))
     (property "Value" "1N4742" (id 1) (at 298.45 210.82 90))
-    (property "Footprint" "BSD_POWER_AMP:D_DO-41_SOD81_P10.16mm_Zener_Horizontal" (id 2) (at 292.1 209.55 0)
+    (property "Footprint" "BSD_POWER_AMP:D_T-1_P10.16mm_Zener_Horizontal" (id 2) (at 292.1 209.55 0)
       (effects (font (size 1.27 1.27)) hide)
     )

Commit message: Update Mon Sep 19 11:44:29 AM WIB 2022
Parts:
- C603, C703: footprint BSD_POWER_AMP:0.0022uF_400V_Vishay_Roederstein_MKT_1822 -> BSD_POWER_AMP:C_Rect_L13.0mm_W4.0mm_P10.00mm_FKS3_FKP3_MKS4
Changed lines of the file:
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@@
     (property "Reference" "C603" (id 0) (at 387.35 60.96 90))
     (property "Value" "2200pF" (id 1) (at 387.35 63.5 90))
-    (property "Footprint" "BSD_POWER_AMP:0.0022uF_400V_Vishay_Roederstein_MKT_1822" (id 2) (at 391.16 58.1152 0)
+    (property "Footprint" "BSD_POWER_AMP:C_Rect_L13.0mm_W4.0mm_P10.00mm_FKS3_FKP3_MKS4" (id 2) (at 391.16 58.1152 0)
       (effects (font (size 1.27 1.27)) hide)
     )
@@
     (property "Reference" "C703" (id 0) (at 387.35 194.31 90))
     (property "Value" "2200pF" (id 1) (at 387.35 196.85 90))
-    (property "Footprint" "BSD_POWER_AMP:0.0022uF_400V_Vishay_Roederstein_MKT_1822" (id 2) (at 383.54 204.1652 0)
-      (effects (font (size 1.27 1.27)) hide)
-    )
+    (property "Footprint" "BSD_POWER_AMP:C_Rect_L13.0mm_W4.0mm_P10.00mm_FKS3_FKP3_MKS4" (id 2) (at 383.54 204.1652 0)
+      (effects (font (size 1.27 1.27)) hide)
+    )

Commit message: Update Mon Sep 19 07:51:54 PM WIB 2022
Connections:
- net REF: now also R401.2; no longer R401.1
- net at C401.2: now also R401.1; no longer R401.2
Changed lines of the file:
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@@
     (pin "3")
   )
-  (symbol (lib_id "Device:R") (at 50.8 107.95 0) (unit 1)
+  (symbol (lib_name "R_46") (lib_id "Device:R") (at 50.8 107.95 0) (unit 1)
     (in_bom yes) (on_board yes)
     (property "Reference" "RG401" (id 0) (at 57.15 105.41 0))
@@
     (pin "1")
   )
-  (symbol (lib_name "R_40") (lib_id "Device:R") (at 63.5 95.25 0) (unit 1)
+  (symbol (lib_name "R_40") (lib_id "Device:R") (at 63.5 95.25 0) (mirror x) (unit 1)
     (in_bom yes) (on_board yes)
     (property "Reference" "R401" (id 0) (at 69.85 92.71 0))
