File: 1300-watts-RMS-for-4-ohms-class-TD-audio-power-amp-DEV-4/POWER-AMP-BLOCK.kicad_sch (KiCad schematic)
At the start: 170 parts, among them Q401 MPSA42, Q402 MPSA42, Q403 MPSA92, Q404 MPSA92, Q405 MJE340, Q406 MJE350, Q407 MJE350, Q408 MJE340, Q409 MJE15032, Q410 MJE15033, Q411 2SC5200, Q412 2SA1943, Q4131 2SC5200, Q4132 2SC5200, Q4133 2SC5200, Q4134 2SC5200, Q4135 2SC5200, Q4136 2SC5200, Q4141 2SA1943, Q4142 2SA1943, Q4143 2SA1943, Q4144 2SA1943, Q4145 2SA1943, Q4146 2SA1943, Q601 2N5401, Q602 MJE340, Q603 MJE340, Q604 MJE15032, Q605 2SC5200, Q606 2N5401, Q607 2N5401, Q608 2N5401, Q609 MJE350, Q610 2N5551, Q611 MJE340, Q701 2N5551, Q702 MJE350, Q703 MJE350, Q704 MJE15033, Q705 2SA1943, Q706 2N5551, Q707 2N5551, Q708 2N5401, Q709 MJE350, Q710 2N5551, Q711 MJE340

Commit message: Update Mon Sep 19 09:45:38 PM WIB 2022
Parts:
- Q411, Q412, Q4131, Q4132, Q4133, Q4134, Q4135, Q4136, Q4141, Q4142, Q4143, Q4144, Q4145, Q4146: footprint BSD_POWER_AMP:TO-264-MIRRORED -> BSD_POWER_AMP:TO-264-3_Vertical_For_Bottom_Layer
Changed lines of the file:
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@@
     (property "Reference" "Q4142" (id 0) (at 247.65 146.05 0))
     (property "Value" "2SA1943" (id 1) (at 247.65 148.59 0))
-    (property "Footprint" "BSD_POWER_AMP:TO-264-MIRRORED" (id 2) (at 243.84 154.94 0)
+    (property "Footprint" "BSD_POWER_AMP:TO-264-3_Vertical_For_Bottom_Layer" (id 2) (at 243.84 154.94 0)
       (effects (font (size 1.27 1.27)) hide)
     )
@@
     (property "Reference" "Q4141" (id 0) (at 234.95 146.05 0))
     (property "Value" "2SA1943" (id 1) (at 234.95 148.59 0))
-    (property "Footprint" "BSD_POWER_AMP:TO-264-MIRRORED" (id 2) (at 231.14 154.94 0)
+    (property "Footprint" "BSD_POWER_AMP:TO-264-3_Vertical_For_Bottom_Layer" (id 2) (at 231.14 154.94 0)
       (effects (font (size 1.27 1.27)) hide)
     )
@@
     (property "Reference" "Q4143" (id 0) (at 260.35 146.05 0))
     (property "Value" "2SA1943" (id 1) (at 260.35 148.59 0))
-    (property "Footprint" "BSD_POWER_AMP:TO-264-MIRRORED" (id 2) (at 256.54 154.94 0)
+    (property "Footprint" "BSD_POWER_AMP:TO-264-3_Vertical_For_Bottom_Layer" (id 2) (at 256.54 154.94 0)
       (effects (font (size 1.27 1.27)) hide)
     )
@@
     (property "Reference" "Q4146" (id 0) (at 298.45 146.05 0))
     (property "Value" "2SA1943" (id 1) (at 298.45 148.59 0))
-    (property "Footprint" "BSD_POWER_AMP:TO-264-MIRRORED" (id 2) (at 294.64 154.94 0)
+    (property "Footprint" "BSD_POWER_AMP:TO-264-3_Vertical_For_Bottom_Layer" (id 2) (at 294.64 154.94 0)
       (effects (font (size 1.27 1.27)) hide)
     )
@@
     (property "Reference" "Q412" (id 0) (at 215.9 157.48 0))
     (property "Value" "2SA1943" (id 1) (at 215.9 160.02 0))
-    (property "Footprint" "BSD_POWER_AMP:TO-264-MIRRORED" (id 2) (at 212.09 161.29 0)
+    (property "Footprint" "BSD_POWER_AMP:TO-264-3_Vertical_For_Bottom_Layer" (id 2) (at 212.09 161.29 0)
       (effects (font (size 1.27 1.27)) hide)
     )
@@
     (property "Reference" "Q4145" (id 0) (at 285.75 146.05 0))
     (property "Value" "2SA1943" (id 1) (at 285.75 148.59 0))
-    (property "Footprint" "BSD_POWER_AMP:TO-264-MIRRORED" (id 2) (at 281.94 154.94 0)
+    (property "Footprint" "BSD_POWER_AMP:TO-264-3_Vertical_For_Bottom_Layer" (id 2) (at 281.94 154.94 0)
       (effects (font (size 1.27 1.27)) hide)
     )
@@
     (property "Reference" "Q4144" (id 0) (at 273.05 146.05 0))
     (property "Value" "2SA1943" (id 1) (at 273.05 148.59 0))
-    (property "Footprint" "BSD_POWER_AMP:TO-264-MIRRORED" (id 2) (at 269.24 154.94 0)
+    (property "Footprint" "BSD_POWER_AMP:TO-264-3_Vertical_For_Bottom_Layer" (id 2) (at 269.24 154.94 0)
       (effects (font (size 1.27 1.27)) hide)
     )
@@
     (property "Reference" "Q4134" (id 0) (at 273.05 118.11 0))
     (property "Value" "2SC5200" (id 1) (at 273.05 120.65 0))
-    (property "Footprint" "BSD_POWER_AMP:TO-264-MIRRORED" (id 2) (at 269.24 111.76 0)
+    (property "Footprint" "BSD_POWER_AMP:TO-264-3_Vertical_For_Bottom_Layer" (id 2) (at 269.24 111.76 0)
       (effects (font (size 1.27 1.27)) hide)
     )
@@
     (property "Reference" "Q4136" (id 0) (at 298.45 118.11 0))
     (property "Value" "2SC5200" (id 1) (at 298.45 120.65 0))
-    (property "Footprint" "BSD_POWER_AMP:TO-264-MIRRORED" (id 2) (at 294.64 111.76 0)
+    (property "Footprint" "BSD_POWER_AMP:TO-264-3_Vertical_For_Bottom_Layer" (id 2) (at 294.64 111.76 0)
       (effects (font (size 1.27 1.27)) hide)
     )
@@
     (property "Reference" "Q4131" (id 0) (at 234.95 118.11 0))
     (property "Value" "2SC5200" (id 1) (at 234.95 120.65 0))
-    (property "Footprint" "BSD_POWER_AMP:TO-264-MIRRORED" (id 2) (at 231.14 111.76 0)
+    (property "Footprint" "BSD_POWER_AMP:TO-264-3_Vertical_For_Bottom_Layer" (id 2) (at 231.14 111.76 0)
       (effects (font (size 1.27 1.27)) hide)
     )
@@
     (property "Reference" "Q4132" (id 0) (at 247.65 118.11 0))
     (property "Value" "2SC5200" (id 1) (at 247.65 120.65 0))
-    (property "Footprint" "BSD_POWER_AMP:TO-264-MIRRORED" (id 2) (at 243.84 111.76 0)
+    (property "Footprint" "BSD_POWER_AMP:TO-264-3_Vertical_For_Bottom_Layer" (id 2) (at 243.84 111.76 0)
       (effects (font (size 1.27 1.27)) hide)
     )
@@
     (property "Reference" "Q411" (id 0) (at 215.9 106.68 0))
     (property "Value" "2SC5200" (id 1) (at 215.9 109.22 0))
-    (property "Footprint" "BSD_POWER_AMP:TO-264-MIRRORED" (id 2) (at 212.09 105.41 0)
+    (property "Footprint" "BSD_POWER_AMP:TO-264-3_Vertical_For_Bottom_Layer" (id 2) (at 212.09 105.41 0)
       (effects (font (size 1.27 1.27)) hide)
     )
@@
     (property "Reference" "Q4133" (id 0) (at 260.35 118.11 0))
     (property "Value" "2SC5200" (id 1) (at 260.35 120.65 0))
-    (property "Footprint" "BSD_POWER_AMP:TO-264-MIRRORED" (id 2) (at 256.54 111.76 0)
+    (property "Footprint" "BSD_POWER_AMP:TO-264-3_Vertical_For_Bottom_Layer" (id 2) (at 256.54 111.76 0)
       (effects (font (size 1.27 1.27)) hide)
     )
@@
     (property "Reference" "Q4135" (id 0) (at 285.75 118.11 0))
     (property "Value" "2SC5200" (id 1) (at 285.75 120.65 0))
-    (property "Footprint" "BSD_POWER_AMP:TO-264-MIRRORED" (id 2) (at 281.94 111.76 0)
+    (property "Footprint" "BSD_POWER_AMP:TO-264-3_Vertical_For_Bottom_Layer" (id 2) (at 281.94 111.76 0)
       (effects (font (size 1.27 1.27)) hide)
     )

Commit message: Update Wed Sep 21 09:39:25 AM WIB 2022
Parts:
- Q605, Q705, XQ6011, XQ6012, XQ7011, XQ7012: footprint BSD_POWER_AMP:TO-264-MIRRORED -> BSD_POWER_AMP:TO-264-3_Vertical_For_Bottom_Layer
Changed lines of the file:
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@@
       (effects (font (size 1.143 1.143) bold))
     )
-    (property "Footprint" "BSD_POWER_AMP:TO-264-MIRRORED" (id 2) (at 358.14 48.26 0)
+    (property "Footprint" "BSD_POWER_AMP:TO-264-3_Vertical_For_Bottom_Layer" (id 2) (at 358.14 48.26 0)
       (effects (font (size 1.27 1.27)) hide)
     )
@@
       (effects (font (size 1.143 1.143) bold))
     )
-    (property "Footprint" "BSD_POWER_AMP:TO-264-MIRRORED" (id 2) (at 345.44 207.01 0)
+    (property "Footprint" "BSD_POWER_AMP:TO-264-3_Vertical_For_Bottom_Layer" (id 2) (at 345.44 207.01 0)
       (effects (font (size 1.27 1.27)) hide)
     )
@@
     (property "Reference" "Q705" (id 0) (at 247.65 195.58 0))
     (property "Value" "2SA1943" (id 1) (at 247.65 198.12 0))
-    (property "Footprint" "BSD_POWER_AMP:TO-264-MIRRORED" (id 2) (at 243.84 199.39 0)
+    (property "Footprint" "BSD_POWER_AMP:TO-264-3_Vertical_For_Bottom_Layer" (id 2) (at 243.84 199.39 0)
       (effects (font (size 1.27 1.27)) hide)
     )
@@
       (effects (font (size 1.143 1.143) bold))
     )
-    (property "Footprint" "BSD_POWER_AMP:TO-264-MIRRORED" (id 2) (at 345.44 41.91 0)
+    (property "Footprint" "BSD_POWER_AMP:TO-264-3_Vertical_For_Bottom_Layer" (id 2) (at 345.44 41.91 0)
       (effects (font (size 1.27 1.27)) hide)
     )
@@
     (property "Reference" "Q605" (id 0) (at 247.65 68.58 0))
     (property "Value" "2SC5200" (id 1) (at 247.65 71.12 0))
-    (property "Footprint" "BSD_POWER_AMP:TO-264-MIRRORED" (id 2) (at 243.84 67.31 0)
+    (property "Footprint" "BSD_POWER_AMP:TO-264-3_Vertical_For_Bottom_Layer" (id 2) (at 243.84 67.31 0)
       (effects (font (size 1.27 1.27)) hide)
     )
@@
       (effects (font (size 1.143 1.143) bold))
     )
-    (property "Footprint" "BSD_POWER_AMP:TO-264-MIRRORED" (id 2) (at 358.14 213.36 0)
-      (effects (font (size 1.27 1.27)) hide)
-    )
+    (property "Footprint" "BSD_POWER_AMP:TO-264-3_Vertical_For_Bottom_Layer" (id 2) (at 358.14 213.36 0)
+      (effects (font (size 1.27 1.27)) hide)
+    )

Commit message: Update Wed Sep 21 11:46:30 AM WIB 2022
Parts:
- RT401: footprint BSD_POWER_AMP:RESISTOR_ROUND_TRIMPOT_STD -> BSD_POWER_AMP:Potentiometer_Runtron_RM-065_Vertical
Changed lines of the file:
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@@
       (effects (font (size 1.27 1.27)) (justify left) hide)
     )
-    (property "Footprint" "BSD_POWER_AMP:RESISTOR_ROUND_TRIMPOT_STD" (id 2) (at 106.172 114.3 90)
+    (property "Footprint" "BSD_POWER_AMP:Potentiometer_Runtron_RM-065_Vertical" (id 2) (at 106.172 114.3 90)
       (effects (font (size 1.27 1.27)) hide)
     )

Commit message: Update Sat Sep 24 09:59:01 AM WIB 2022
Connections:
- net VMOUT: now also L401.1; no longer L401.2
- net VPOUT: now also L401.2; no longer L401.1
Changed lines of the file:
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@@
   (title_block
     (title "1300 WATTS RMS CLASS-TD\\nAUDIO POWER AMPLIFIER\\nFOR 4-OHMS LOUDSPEAKER")
-    (date "2022-09-14")
+    (date "2022-09-24")
     (company "BSD POWER AMP")
   )
@@
     (pin "2")
   )
-  (symbol (lib_id "Device:L_Small") (at 304.8 127 0) (unit 1)
+  (symbol (lib_id "Device:L_Small") (at 304.8 127 0) (mirror x) (unit 1)
     (in_bom yes) (on_board yes)
     (property "Reference" "L401" (id 0) (at 311.15 125.73 0))

Commit message: Update Sat Sep 24 07:18:10 PM WIB 2022
Parts:
- D602, D610, D702, D709, D711: Spice_Model 1N4007 -> BAV21
Changed lines of the file:
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@@
       (effects (font (size 1.27 1.27)) hide)
     )
-    (property "Spice_Model" "1N4007" (id 5) (at 255.27 208.28 0)
+    (property "Spice_Model" "BAV21" (id 5) (at 255.27 208.28 0)
       (effects (font (size 1.27 1.27)) hide)
     )
@@
       (effects (font (size 1.27 1.27)) hide)
     )
-    (property "Spice_Model" "1N4007" (id 5) (at 297.18 214.63 0)
+    (property "Spice_Model" "BAV21" (id 5) (at 297.18 214.63 0)
       (effects (font (size 1.27 1.27)) hide)
     )
@@
       (effects (font (size 1.27 1.27)) hide)
     )
-    (property "Spice_Model" "1N4007" (id 5) (at 134.62 179.07 0)
+    (property "Spice_Model" "BAV21" (id 5) (at 134.62 179.07 0)
       (effects (font (size 1.27 1.27)) hide)
     )
@@
       (effects (font (size 1.27 1.27)) hide)
     )
-    (property "Spice_Model" "1N4007" (id 5) (at 255.27 64.77 0)
+    (property "Spice_Model" "BAV21" (id 5) (at 255.27 64.77 0)
       (effects (font (size 1.27 1.27)) hide)
     )
@@
       (effects (font (size 1.27 1.27)) hide)
     )
-    (property "Spice_Model" "1N4007" (id 5) (at 134.62 90.17 0)
-      (effects (font (size 1.27 1.27)) hide)
-    )
+    (property "Spice_Model" "BAV21" (id 5) (at 134.62 90.17 0)
+      (effects (font (size 1.27 1.27)) hide)
+    )

Commit message: Update Sun Sep 25 11:43:47 AM WIB 2022
Parts:
- CNT402: value Solder Tab 6.3 mm -> PinHeader_1x01_P2.54mm_Vertical
- CNT403, CNT404, CNT405: value Solder Tab 6.3 mm -> Solder_Tab_W6.35mm_P5.08mm; footprint BSD_POWER_AMP:SOLDER-TAB-6.3-mm -> BSD_POWER_AMP:Solder_Tab_W6.35mm_P5.08mm
Changed lines of the file:
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@@
     (in_bom yes) (on_board yes)
     (property "Reference" "CNT403" (id 0) (at 38.1 22.86 0))
-    (property "Value" "Solder Tab 6.3 mm" (id 1) (at 38.1 15.24 0)
+    (property "Value" "Solder_Tab_W6.35mm_P5.08mm" (id 1) (at 38.1 15.24 0)
       (effects (font (size 1.27 1.27)) hide)
     )
-    (property "Footprint" "BSD_POWER_AMP:SOLDER-TAB-6.3-mm" (id 2) (at 38.1 19.05 0)
+    (property "Footprint" "BSD_POWER_AMP:Solder_Tab_W6.35mm_P5.08mm" (id 2) (at 38.1 19.05 0)
       (effects (font (size 1.27 1.27)) hide)
     )
@@
     (in_bom yes) (on_board yes)
     (property "Reference" "CNT405" (id 0) (at 38.1 168.91 0))
-    (property "Value" "Solder Tab 6.3 mm" (id 1) (at 38.1 161.29 0)
+    (property "Value" "Solder_Tab_W6.35mm_P5.08mm" (id 1) (at 38.1 161.29 0)
       (effects (font (size 1.27 1.27)) hide)
     )
-    (property "Footprint" "BSD_POWER_AMP:SOLDER-TAB-6.3-mm" (id 2) (at 38.1 165.1 0)
+    (property "Footprint" "BSD_POWER_AMP:Solder_Tab_W6.35mm_P5.08mm" (id 2) (at 38.1 165.1 0)
       (effects (font (size 1.27 1.27)) hide)
     )
@@
     (in_bom yes) (on_board yes)
     (property "Reference" "CNT404" (id 0) (at 38.1 243.84 0))
-    (property "Value" "Solder Tab 6.3 mm" (id 1) (at 38.1 243.84 0)
+    (property "Value" "Solder_Tab_W6.35mm_P5.08mm" (id 1) (at 38.1 243.84 0)
       (effects (font (size 1.27 1.27)) hide)
     )
-    (property "Footprint" "BSD_POWER_AMP:SOLDER-TAB-6.3-mm" (id 2) (at 38.1 247.65 0)
+    (property "Footprint" "BSD_POWER_AMP:Solder_Tab_W6.35mm_P5.08mm" (id 2) (at 38.1 247.65 0)
       (effects (font (size 1.27 1.27)) hide)
     )
@@
     (in_bom yes) (on_board yes)
     (property "Reference" "CNT402" (id 0) (at 38.1 105.41 0))
-    (property "Value" "Solder Tab 6.3 mm" (id 1) (at 38.1 97.79 0)
+    (property "Value" "PinHeader_1x01_P2.54mm_Vertical" (id 1) (at 38.1 97.79 0)
       (effects (font (size 1.27 1.27)) hide)
     )
