File: 1300-watts-RMS-for-4-ohms-class-TD-audio-power-amp-DEV-5/POWER-AMP-BLOCK.kicad_sch (KiCad schematic)
At the start: 183 parts, among them Q401 MJE350, Q402 MJE340, Q403 MJE340, Q404 MJE350, Q405 MJE350, Q406 MJE340, Q407 MJE350, Q408 MJE15032, Q409 MJE15033, Q410 2SC5200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

Commit message: Update Tue Oct 11 06:15:54 PM WIB 2022
Parts:
- R401: value 820 -> 560
Other:
- moved on the sheet: C401, C402, C403, C404, C405, C406, C410, C411, CNT401, D401, D402, D403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
