File: 1300-watts-RMS-for-4-ohms-class-TD-audio-power-amp-DEV-6/POWER-AMP-BLOCK.kicad_sch (KiCad schematic)
At the start: 184 parts, among them Q401 MJE350, Q402 MJE340, Q403 MJE340, Q404 MJE350, Q405 MJE350, Q406 MJE340, Q407 MJE350, Q408 MJE15032, Q409 MJE15033, Q410 2SC5200, Q411 2SA1943, Q4121 2SC5200, Q4122 2SC5200, Q4123 2SC5200, Q4124 2SC5200, Q4125 2SC5200, Q4126 2SC5200, Q4131 2SA1943, Q4132 2SA1943, Q4133 2SA1943, Q4134 2SA1943, Q4135 2SA1943, Q4136 2SA1943, Q601 2N5401, Q602 MJE340, Q603 MJE340, Q604 MJE15032, Q605 2SC5200, Q606 2N5401, Q607 2N5401, Q608 2N5401, Q609 MJE350, Q610 2N5551, Q611 MJE340, Q701 2N5551, Q702 MJE350, Q703 MJE350, Q704 MJE15033, Q705 2SA1943, Q706 2N5551, Q707 2N5551, Q708 2N5401, Q709 MJE350, Q710 2N5551, Q711 MJE340, U401 NE5534

Commit message: Update Wed Oct 12 04:03:10 AM WIB 2022
Parts:
- C404: value 33pF -> 27pF
Changed lines of the file:
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@@
     (in_bom yes) (on_board yes)
     (property "Reference" "C404" (id 0) (at 83.82 111.76 90))
-    (property "Value" "33pF" (id 1) (at 83.82 114.3 90))
+    (property "Value" "27pF" (id 1) (at 83.82 114.3 90))
     (property "Footprint" "BSD_POWER_AMP:C_Disc_D8.0mm_W5.0mm_P10.00mm" (id 2) (at 87.63 119.6848 0)
       (effects (font (size 1.27 1.27)) hide)
