File: LP-SERIES-DEV-1/POWER-AMP-BLOCK.kicad_sch (KiCad schematic)
At the start: 122 parts, among them Q401 MJE350, Q402 MJE340, Q403 MJE340, Q404 MJE350, Q405 MJE350, Q406 MJE340, Q407 MJE350, Q408 MJE15032, Q409 MJE15033, Q410 2SC5200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

Commit message: Update Sat Oct 22 04:32:29 AM WIB 2022
Parts:
- C402, C404, C405, C407: footprint Capacitor_THT:C_Disc_D8.0mm_W5.0mm_P5.00mm -> Capacitor_THT:C_Disc_D8.0mm_W2.5mm_P5.00mm
- D501, D504, D507, D601, D604, D701: footprint BSD_POWER_AMP:D_T-1_P2.54mm_Vertical_KathodeUp -> BSD_POWER_AMP:D_DO-35_SOD27_P5.08mm_Vertical_KathodeUp
- R405: footprint Resistor_THT:R_Axial_DIN0207_L6.3mm_D2.5mm_P2.54mm_Vertical -> Resistor_THT:R_Axial_DIN0207_L6.3mm_D2.5mm_P5.08mm_Vertical
Connections:
- net +15V: now also CNT402.1 (Pin_1); no longer CNT402.3 (Pin_3)
- net -15V: now also CNT402.3 (Pin_3); no longer CNT402.1 (Pin_1)
- net VASGCTLN: now also R415.2, R416.1; no longer R415.1, R416.2
- net VASGCTLP: now also R412.2; no longer R412.1
- net VASN: now also R416.2; no longer R416.1
- net VASP: now also R412.1; no longer R412.2
- net at D412.2 (K): now also R415.1; no longer R415.2
Other:
- note added: "+15 GND -15"
- note removed: "-15 GND +15"
- moved on the sheet: R412, R415, R416
Changed lines of the file:
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@@
   (title_block
     (title "290 WATTS RMS CLASS-H\\nAUDIO POWER AMPLIFIER\\nFOR 4-OHMS LOUDSPEAKER")
-    (date "2022-10-21")
+    (date "2022-10-22")
     (company "BSD POWER AMP")
   )
@@
     (effects (font (size 1.397 1.397)) (justify left bottom))
   )
-  (text "-15\nGND\n+15" (at 51.435 142.621 0)
+  (text "+15\nGND\n-15" (at 51.435 142.621 0)
     (effects (font (size 1.27 1.27)) (justify left bottom))
   )
@@
     )
   )
-  (global_label "+15V" (shape output) (at 76.2 142.24 0) (fields_autoplaced)
+  (global_label "-15V" (shape output) (at 76.2 142.24 0) (fields_autoplaced)
     (effects (font (size 1.27 1.27)) (justify left))
-    (property "Intersheet References" "${INTERSHEET_REFS}" (id 0) (at 83.5026 142.1606 0)
+    (property "Intersheet References" "${INTERSHEET_REFS}" (id 0) (at 83.6931 142.1606 0)
       (effects (font (size 1.27 1.27)) (justify left) hide)
     )
@@
     )
   )
-  (global_label "-15V" (shape output) (at 76.2 137.16 0) (fields_autoplaced)
+  (global_label "+15V" (shape output) (at 76.2 137.16 0) (fields_autoplaced)
     (effects (font (size 1.27 1.27)) (justify left))
-    (property "Intersheet References" "${INTERSHEET_REFS}" (id 0) (at 83.5026 137.0806 0)
+    (property "Intersheet References" "${INTERSHEET_REFS}" (id 0) (at 83.6931 137.0806 0)
       (effects (font (size 1.27 1.27)) (justify left) hide)
     )
@@
     (pin "2")
   )
-  (symbol (lib_name "R_32") (lib_id "Device:R") (at 171.45 184.15 270) (mirror x) (unit 1)
+  (symbol (lib_name "R_2") (lib_id "Device:R") (at 171.45 184.15 90) (unit 1)
     (in_bom yes) (on_board yes)
     (property "Reference" "R415" (id 0) (at 171.45 175.26 90))
@@
     (property "Reference" "C407" (id 0) (at 203.2 187.96 90))
     (property "Value" "82pF" (id 1) (at 203.2 190.5 90))
-    (property "Footprint" "Capacitor_THT:C_Disc_D8.0mm_W5.0mm_P5.00mm" (id 2) (at 199.39 195.8848 0)
+    (property "Footprint" "Capacitor_THT:C_Disc_D8.0mm_W2.5mm_P5.00mm" (id 2) (at 199.39 195.8848 0)
       (effects (font (size 1.27 1.27)) hide)
     )
@@
     (property "Reference" "C404" (id 0) (at 140.97 118.11 90))
     (property "Value" "33pF" (id 1) (at 140.97 120.65 90))
-    (property "Footprint" "Capacitor_THT:C_Disc_D8.0mm_W5.0mm_P5.00mm" (id 2) (at 144.78 126.0348 0)
+    (property "Footprint" "Capacitor_THT:C_Disc_D8.0mm_W2.5mm_P5.00mm" (id 2) (at 144.78 126.0348 0)
       (effects (font (size 1.27 1.27)) hide)
     )
@@
     (property "Reference" "C402" (id 0) (at 95.25 149.86 90))
     (property "Value" "220pF" (id 1) (at 95.25 152.4 90))
-    (property "Footprint" "Capacitor_THT:C_Disc_D8.0mm_W5.0mm_P5.00mm" (id 2) (at 99.06 145.0848 0)
+    (property "Footprint" "Capacitor_THT:C_Disc_D8.0mm_W2.5mm_P5.00mm" (id 2) (at 99.06 145.0848 0)
       (effects (font (size 1.27 1.27)) hide)
     )
@@
     (property "Reference" "D507" (id 0) (at 304.8 87.63 90))
     (property "Value" "1N4742" (id 1) (at 304.8 90.17 90))
-    (property "Footprint" "BSD_POWER_AMP:D_T-1_P2.54mm_Vertical_KathodeUp" (id 2) (at 298.45 88.9 0)
+    (property "Footprint" "BSD_POWER_AMP:D_DO-35_SOD27_P5.08mm_Vertical_KathodeUp" (id 2) (at 298.45 88.9 0)
       (effects (font (size 1.27 1.27)) hide)
     )
@@
     (property "Reference" "D701" (id 0) (at 317.5 121.92 90))
     (property "Value" "1N4753" (id 1) (at 317.5 124.46 90))
-    (property "Footprint" "BSD_POWER_AMP:D_T-1_P2.54mm_Vertical_KathodeUp" (id 2) (at 311.15 123.19 0)
+    (property "Footprint" "BSD_POWER_AMP:D_DO-35_SOD27_P5.08mm_Vertical_KathodeUp" (id 2) (at 311.15 123.19 0)
       (effects (font (size 1.27 1.27)) hide)
     )
@@
     (property "Reference" "D601" (id 0) (at 241.3 189.23 90))
     (property "Value" "1N4736" (id 1) (at 241.3 191.77 90))
-    (property "Footprint" "BSD_POWER_AMP:D_T-1_P2.54mm_Vertical_KathodeUp" (id 2) (at 234.95 190.5 0)
+    (property "Footprint" "BSD_POWER_AMP:D_DO-35_SOD27_P5.08mm_Vertical_KathodeUp" (id 2) (at 234.95 190.5 0)
       (effects (font (size 1.27 1.27)) hide)
     )
@@
     (pin "8")
   )
-  (symbol (lib_name "R_18") (lib_id "Device:R") (at 184.15 95.25 90) (unit 1)
+  (symbol (lib_name "R_5") (lib_id "Device:R") (at 184.15 95.25 270) (mirror x) (unit 1)
     (in_bom yes) (on_board yes)
     (property "Reference" "R412" (id 0) (at 184.15 99.06 90))
@@
     (property "Reference" "D501" (id 0) (at 241.3 100.33 90))
     (property "Value" "1N4736" (id 1) (at 241.3 102.87 90))
-    (property "Footprint" "BSD_POWER_AMP:D_T-1_P2.54mm_Vertical_KathodeUp" (id 2) (at 234.95 101.6 0)
+    (property "Footprint" "BSD_POWER_AMP:D_DO-35_SOD27_P5.08mm_Vertical_KathodeUp" (id 2) (at 234.95 101.6 0)
       (effects (font (size 1.27 1.27)) hide)
     )
@@
     (property "Reference" "C405" (id 0) (at 203.2 86.36 90))
     (property "Value" "82pF" (id 1) (at 203.2 88.9 90))
-    (property "Footprint" "Capacitor_THT:C_Disc_D8.0mm_W5.0mm_P5.00mm" (id 2) (at 199.39 81.5848 0)
+    (property "Footprint" "Capacitor_THT:C_Disc_D8.0mm_W2.5mm_P5.00mm" (id 2) (at 199.39 81.5848 0)
       (effects (font (size 1.27 1.27)) hide)
     )
@@
     (property "Reference" "R405" (id 0) (at 120.65 187.96 0))
     (property "Value" "10" (id 1) (at 120.65 190.5 0))
-    (property "Footprint" "Resistor_THT:R_Axial_DIN0207_L6.3mm_D2.5mm_P2.54mm_Vertical" (id 2) (at 112.522 190.5 90)
+    (property "Footprint" "Resistor_THT:R_Axial_DIN0207_L6.3mm_D2.5mm_P5.08mm_Vertical" (id 2) (at 112.522 190.5 90)
       (effects (font (size 1.27 1.27)) hide)
     )
@@
     (pin "2")
   )
-  (symbol (lib_name "R_28") (lib_id "Device:R") (at 184.15 184.15 270) (mirror x) (unit 1)
+  (symbol (lib_name "R_28") (lib_id "Device:R") (at 184.15 184.15 90) (unit 1)
     (in_bom yes) (on_board yes)
     (property "Reference" "R416" (id 0) (at 184.15 175.26 90))
@@
     (property "Reference" "D504" (id 0) (at 266.7 68.58 90))
     (property "Value" "1N4749" (id 1) (at 266.7 71.12 90))
-    (property "Footprint" "BSD_POWER_AMP:D_T-1_P2.54mm_Vertical_KathodeUp" (id 2) (at 260.35 69.85 0)
+    (property "Footprint" "BSD_POWER_AMP:D_DO-35_SOD27_P5.08mm_Vertical_KathodeUp" (id 2) (at 260.35 69.85 0)
       (effects (font (size 1.27 1.27)) hide)
     )
@@
     (property "Reference" "D604" (id 0) (at 304.8 208.28 90))
     (property "Value" "1N4742" (id 1) (at 304.8 210.82 90))
-    (property "Footprint" "BSD_POWER_AMP:D_T-1_P2.54mm_Vertical_KathodeUp" (id 2) (at 298.45 209.55 0)
+    (property "Footprint" "BSD_POWER_AMP:D_DO-35_SOD27_P5.08mm_Vertical_KathodeUp" (id 2) (at 298.45 209.55 0)
       (effects (font (size 1.27 1.27)) hide)
     )
@@
     (pin "2")
   )
-  (symbol (lib_name "R_32") (lib_id "Device:R") (at 171.45 95.25 270) (mirror x) (unit 1)
+  (symbol (lib_name "R_6") (lib_id "Device:R") (at 171.45 95.25 270) (mirror x) (unit 1)
     (in_bom yes) (on_board yes)
     (property "Reference" "R411" (id 0) (at 171.45 86.36 90))

Commit message: Update Sun Oct 23 04:54:01 PM WIB 2022
Parts:
- C403: footprint Capacitor_THT:CP_Radial_D10.0mm_P5.00mm -> Capacitor_THT:CP_Radial_D8.0mm_P5.00mm
- C501: footprint Capacitor_THT:CP_Radial_D5.0mm_P2.50mm -> Capacitor_THT:CP_Radial_D6.3mm_P2.50mm
- L401: footprint BSD_POWER_AMP:INDUCTOR_AIR_CORE_3uH_D600mils_L750mils -> BSD_POWER_AMP:INDUCTOR_AIR_CORE_1uH
- RT401: footprint Potentiometer_THT:Potentiometer_Runtron_RM-065_Vertical -> BSD_POWER_AMP:Potentiometer_Runtron_RM-065_Vertical_STD
Connections:
- net VBT: now reaches R421.1, R422.2, RT401.2
- net VSB: now reaches Q407.2 (B), R419.1, R420.2, R421.2
- net L_GCTL: now reaches Q604.3 (E), Q605.3 (E), XQ601.2 (G)
- net H_GCTL: now reaches Q503.3 (E), Q504.3 (E), XQ501.2 (G)
Other:
- moved on the sheet: Q407

Commit message: Update Sun Oct 23 05:22:13 PM WIB 2022
Parts:
- L401: symbol Device:L_Small -> Device:L
Changed lines of the file:
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@@
   (title_block
     (title "290 WATTS RMS CLASS-H\\nAUDIO POWER AMPLIFIER\\nFOR 4-OHMS LOUDSPEAKER")
-    (date "2022-10-22")
+    (date "2022-10-23")
     (company "BSD POWER AMP")
   )
@@
   (junction (at 203.2 139.7) (diameter 0) (color 0 0 0 0)
   )
-  (junction (at 304.8 139.7) (diameter 0) (color 0 0 0 0)
-  )
   (junction (at 311.15 107.95) (diameter 0) (color 0 0 0 0)
   )
@@
   (junction (at 285.75 63.5) (diameter 0) (color 0 0 0 0)
   )
+  (junction (at 304.8 139.7) (diameter 0) (color 0 0 0 0)
+  )
   (junction (at 88.9 146.05) (diameter 0) (color 0 0 0 0)
   )
@@
     (stroke (width 0) (type default) (color 0 0 0 0))
   )
-  (wire (pts (xy 320.04 139.7) (xy 344.17 139.7))
-    (stroke (width 0) (type default) (color 0 0 0 0))
-  )
   (wire (pts (xy 323.85 107.95) (xy 323.85 110.49))
     (stroke (width 0) (type default) (color 0 0 0 0))
@@
     (stroke (width 0) (type default) (color 0 0 0 0))
   )
-  (wire (pts (xy 304.8 139.7) (xy 314.96 139.7))
-    (stroke (width 0) (type default) (color 0 0 0 0))
-  )
   (polyline (pts (xy 52.07 57.15) (xy 62.23 57.15))
     (stroke (width 0) (type solid) (color 0 0 0 0))
@@
     (stroke (width 0) (type default) (color 0 0 0 0))
   )
+  (wire (pts (xy 321.31 139.7) (xy 344.17 139.7))
+    (stroke (width 0) (type default) (color 0 0 0 0))
+  )
   (wire (pts (xy 222.25 158.75) (xy 273.05 158.75))
     (stroke (width 0) (type default) (color 0 0 0 0))
@@
     (stroke (width 0) (type default) (color 0 0 0 0))
   )
+  (wire (pts (xy 304.8 139.7) (xy 313.69 139.7))
+    (stroke (width 0) (type default) (color 0 0 0 0))
+  )
   (wire (pts (xy 209.55 165.1) (xy 209.55 156.21))
     (stroke (width 0) (type default) (color 0 0 0 0))
@@
     )
   )
-  (global_label "VPOUT" (shape passive) (at 330.2 139.7 270) (fields_autoplaced)
+  (global_label "VPOUT" (shape passive) (at 331.47 139.7 270) (fields_autoplaced)
     (effects (font (size 1.27 1.27)) (justify right))
-    (property "Intersheet References" "${INTERSHEET_REFS}" (id 0) (at 330.1206 148.1002 90)
+    (property "Intersheet References" "${INTERSHEET_REFS}" (id 0) (at 331.3906 148.1002 90)
       (effects (font (size 1.27 1.27)) (justify right) hide)
     )
@@
     (pin "2")
   )
-  (symbol (lib_id "Device:L_Small") (at 317.5 139.7 90) (mirror x) (unit 1)
+  (symbol (lib_id "Device:L") (at 317.5 139.7 90) (mirror x) (unit 1)
     (in_bom yes) (on_board yes)
     (property "Reference" "L401" (id 0) (at 317.5 146.05 90))
