File: LP-SERIES-DEV-1/POWER-AMP-BLOCK.kicad_sch (KiCad schematic)
At the start: 122 parts, among them Q401 MJE350, Q402 MJE340, Q403 MJE340, Q404 MJE350, Q405 MJE350, Q406 MJE340, Q407 MJE350, Q408 MJE15032, Q409 MJE15033, Q410 2SC5200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

Commit message: Update Mon Oct 24 02:14:06 PM WIB 2022
Parts:
- D501, D504, D507, D601, D604: footprint BSD_POWER_AMP:D_DO-35_SOD27_P5.08mm_Vertical_KathodeUp -> BSD_POWER_AMP:D_T-1_DO-35_SOD27_P5.08mm_Vertical_KathodeUp
Changed lines of the file:
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@@
     (property "Reference" "D507" (id 0) (at 304.8 87.63 90))
     (property "Value" "1N4742" (id 1) (at 304.8 90.17 90))
-    (property "Footprint" "BSD_POWER_AMP:D_DO-35_SOD27_P5.08mm_Vertical_KathodeUp" (id 2) (at 298.45 88.9 0)
+    (property "Footprint" "BSD_POWER_AMP:D_T-1_DO-35_SOD27_P5.08mm_Vertical_KathodeUp" (id 2) (at 298.45 88.9 0)
       (effects (font (size 1.27 1.27)) hide)
     )
@@
     (property "Reference" "D601" (id 0) (at 241.3 189.23 90))
     (property "Value" "1N4736" (id 1) (at 241.3 191.77 90))
-    (property "Footprint" "BSD_POWER_AMP:D_DO-35_SOD27_P5.08mm_Vertical_KathodeUp" (id 2) (at 234.95 190.5 0)
+    (property "Footprint" "BSD_POWER_AMP:D_T-1_DO-35_SOD27_P5.08mm_Vertical_KathodeUp" (id 2) (at 234.95 190.5 0)
       (effects (font (size 1.27 1.27)) hide)
     )
@@
     (property "Reference" "D501" (id 0) (at 241.3 100.33 90))
     (property "Value" "1N4736" (id 1) (at 241.3 102.87 90))
-    (property "Footprint" "BSD_POWER_AMP:D_DO-35_SOD27_P5.08mm_Vertical_KathodeUp" (id 2) (at 234.95 101.6 0)
+    (property "Footprint" "BSD_POWER_AMP:D_T-1_DO-35_SOD27_P5.08mm_Vertical_KathodeUp" (id 2) (at 234.95 101.6 0)
       (effects (font (size 1.27 1.27)) hide)
     )
@@
     (property "Reference" "D504" (id 0) (at 266.7 68.58 90))
     (property "Value" "1N4749" (id 1) (at 266.7 71.12 90))
-    (property "Footprint" "BSD_POWER_AMP:D_DO-35_SOD27_P5.08mm_Vertical_KathodeUp" (id 2) (at 260.35 69.85 0)
+    (property "Footprint" "BSD_POWER_AMP:D_T-1_DO-35_SOD27_P5.08mm_Vertical_KathodeUp" (id 2) (at 260.35 69.85 0)
       (effects (font (size 1.27 1.27)) hide)
     )
@@
     (property "Reference" "D604" (id 0) (at 304.8 208.28 90))
     (property "Value" "1N4742" (id 1) (at 304.8 210.82 90))
-    (property "Footprint" "BSD_POWER_AMP:D_DO-35_SOD27_P5.08mm_Vertical_KathodeUp" (id 2) (at 298.45 209.55 0)
-      (effects (font (size 1.27 1.27)) hide)
-    )
+    (property "Footprint" "BSD_POWER_AMP:D_T-1_DO-35_SOD27_P5.08mm_Vertical_KathodeUp" (id 2) (at 298.45 209.55 0)
+      (effects (font (size 1.27 1.27)) hide)
+    )
